File: motherboard-2PIECES.sch (KiCad schematic (older format))
At the start: 11 parts, among them X1 MEC1, X2 MEC1, X3 MEC1, X4 MEC1, Y1 MEC1, Y2 MEC1, Y3 MEC1, Y4 MEC1

Commit message: Cleanup: Obviously the temporary files were newer
Parts:
- added Linker? (x2), LinkerToTB?: CONN_20X2, symbol CONN_20X2
Connections:
- net +AIN1: now also LinkerToTB?.10 (P10); no longer LinkerToTB1.31 (P31)
- net +AIN2: now also Linker?.2 (P2), LinkerToTB?.2 (P2); no longer Linker1.39 (P39), LinkerToTB1.39 (P39)
- net -AIN1: now also LinkerToTB?.12 (P12); no longer LinkerToTB1.32 (P32)
- net -AIN2: now also Linker?.4 (P4), LinkerToTB?.4 (P4); no longer Linker1.40 (P40), LinkerToTB1.40 (P40)
- net AREF: now also Linker?.9 (P9), LinkerToTB?.7 (P7); no longer Linker1.33 (P33), LinkerToTB1.33 (P33)
- net CAL: now also Linker?.12 (P12), LinkerToTB?.15 (P15); no longer Linker1.30 (P30), LinkerToTB1.30 (P30)
- net CS: now also Linker?.27 (P27), LinkerToTB?.27 (P27); no longer Linker1.13 (P13), LinkerToTB1.13 (P13)
- net CS2: now also Linker?.25, LinkerToTB?.25; no longer Linker1.15 (P15), LinkerToTB1.15 (P15)
- net GND: now also Linker?.1 (P1), Linker?.3 (P3), Linker?.5 (P5), Linker?.5 (P5), Linker?.8 (P8), LinkerToTB?.1 (P1), LinkerToTB?.11 (P11), LinkerToTB?.13 (P13), LinkerToTB?.3 (P3), LinkerToTB?.5 (P5), LinkerToTB?.9 (P9); no longer Linker1.35 (P35), Linker2.35 (P35), LinkerToTB1.35 (P35)
- net IFB: now also Linker?.20 (P20), LinkerToTB?.20 (P20); no longer Linker1.22 (P22), LinkerToTB1.22 (P22)
- net IS1: now also Linker?.21 (P21), LinkerToTB?.21 (P21); no longer Linker1.19 (P19), LinkerToTB1.19 (P19)
- net IS2: now also Linker?.24 (P24), LinkerToTB?.24 (P24); no longer Linker1.18 (P18), LinkerToTB1.18 (P18)
- net LE: now also Linker?.19 (P19), LinkerToTB?.19 (P19); no longer Linker1.21 (P21), LinkerToTB1.21 (P21)
- net R12: now also Linker?.28 (P28), LinkerToTB?.28 (P28); no longer Linker1.14 (P14), LinkerToTB1.14 (P14)
- net RBI: now also Linker?.6 (P6), LinkerToTB?.32 (P32); no longer Linker1.37 (P37), LinkerToTB1.10 (P10)
- net RBO1: now also LinkerToTB?.8 (P8); no longer LinkerToTB1.34 (P34)
- net RBO2: now also Linker?.7 (P7), LinkerToTB?.6 (P6); no longer Linker1.38 (P38), LinkerToTB1.38 (P38)
- net RESET: now also Linker?.22 (P22), LinkerToTB?.22 (P22); no longer Linker1.20 (P20), LinkerToTB1.20 (P20)
- net RPHI1: now also Linker?.31 (P31), LinkerToTB?.31 (P31); no longer Linker1.9 (P9), LinkerToTB1.9 (P9)
- net RPHI2: now also Linker?.34 (P34), LinkerToTB?.34 (P34); no longer Linker1.8 (P8), LinkerToTB1.8 (P8)
- net SBI: now also Linker?.13 (P13), LinkerToTB?.16 (P16); no longer Linker1.27 (P27), LinkerToTB1.27 (P27)
- net SEB: now also Linker?.11 (P11), LinkerToTB?.14 (P14); no longer Linker1.29 (P29), LinkerToTB1.29 (P29)
- net SPHI1: now also Linker?.15 (P15), LinkerToTB?.17 (P17); no longer Linker1.25, LinkerToTB1.25
- net SPHI2: now also Linker?.17 (P17), LinkerToTB?.18 (P18); no longer Linker1.23 (P23), LinkerToTB1.23 (P23)
- net SR: now also Linker?.23 (P23), LinkerToTB?.23 (P23); no longer Linker1.17 (P17), LinkerToTB1.17 (P17)
- net Vana: now also Linker?.35 (P35), LinkerToTB?.35 (P35); no longer Linker1.5 (P5), LinkerToTB1.5 (P5)
- net Vbias: now also Linker?.39 (P39), LinkerToTB?.39 (P39); no longer Linker1.1 (P1), LinkerToTB1.1 (P1)
- net Vdig: now also Linker?.36 (P36), LinkerToTB?.36 (P36); no longer Linker1.6 (P6), LinkerToTB1.6 (P6)
- net Vthresh: now also Linker?.30 (P30), LinkerToTB?.30 (P30); no longer Linker1.12 (P12), LinkerToTB1.12 (P12)
- net _+AIN2: now also Linker?.1 (P1); no longer Linker2.39 (P39)
- net _-AIN2: now also Linker?.2 (P2); no longer Linker2.40 (P40)
- net _AREF: now also Linker?.7 (P7); no longer Linker2.33 (P33)
- net _CAL: now also Linker?.12 (P12); no longer Linker2.30 (P30)
- net _CS: now also Linker?.27 (P27); no longer Linker2.13 (P13)
- net _CS2: now also Linker?.25; no longer Linker2.15 (P15)
- net _IFB: now also Linker?.20 (P20); no longer Linker2.22 (P22)
- net _IS1: now also Linker?.21 (P21); no longer Linker2.19 (P19)
- net _IS2: now also Linker?.24 (P24); no longer Linker2.18 (P18)
- net _LE: now also Linker?.19 (P19); no longer Linker2.21 (P21)
- net _R12: now also Linker?.28 (P28); no longer Linker2.14 (P14)
- net _RBI: now also Linker?.3 (P3); no longer Linker2.37 (P37)
- net _RBO2: now also Linker?.4 (P4); no longer Linker2.38 (P38)
- net _RESET: now also Linker?.22 (P22); no longer Linker2.20 (P20)
- net _RPHI1: now also Linker?.31 (P31); no longer Linker2.9 (P9)
- net _RPHI2: now also Linker?.34 (P34); no longer Linker2.8 (P8)
- net _SBI: now also Linker?.13 (P13); no longer Linker2.27 (P27)
- net _SEB: now also Linker?.11 (P11); no longer Linker2.29 (P29)
- net _SPHI1: now also Linker?.15 (P15); no longer Linker2.25
- net _SPHI2: now also Linker?.17 (P17); no longer Linker2.23 (P23)
- net _SR: now also Linker?.23 (P23); no longer Linker2.17 (P17)
- net _Vana: now also Linker?.35 (P35); no longer Linker2.5 (P5)
- net _Vbias: now also Linker?.39 (P39); no longer Linker2.1 (P1)
- net _Vdig: now also Linker?.36 (P36); no longer Linker2.6 (P6)
- net _Vthresh: now also Linker?.30 (P30); no longer Linker2.12 (P12)
- no-connect marks 71 -> 63
Other:
- moved on the sheet: Linker1, Linker2, LinkerToTB1
Changed lines of the file:
@@
-EESchema Schematic File Version 2  date 5/15/2012 11:50:02 AM
+EESchema Schematic File Version 2  date 8/21/2012 12:30:24 PM
 LIBS:power
 LIBS:device
@@
 Sheet 1 1
 Title ""
-Date "15 may 2012"
+Date "21 aug 2012"
 Rev ""
 Comp ""
@@
 Comment4 ""
 $EndDescr
-NoConn ~ 9700 9300
-NoConn ~ 23000 9200
-NoConn ~ 23000 9100
-NoConn ~ 22200 9100
-NoConn ~ 22200 8900
-NoConn ~ 22200 8700
-NoConn ~ 23000 8500
-NoConn ~ 23000 8100
-NoConn ~ 23000 8000
-NoConn ~ 23000 7900
-NoConn ~ 23000 7500
-NoConn ~ 22200 7400
+$Comp
+L CONN_20X2 Linker?
+U 1 1 5033625F
+P 9300 8450
+F 0 "Linker?" H 9300 9500 60  0000 C CNN
+F 1 "CONN_20X2" V 9300 8450 50  0000 C CNN
+	1    9300 8450
+	1    0    0    -1
+$EndComp
+Connection ~ 12600 6450
+Wire Wire Line
+	12600 6450 12600 7700
+Wire Wire Line
+	12600 7700 12700 7700
+Wire Wire Line
+	12200 6450 12700 6450
+Wire Wire Line
+	12700 6450 12700 7500
+Wire Wire Line
+	23100 5900 13450 5900
+Wire Wire Line
+	23150 6050 13550 6050
+Wire Wire Line
+	12700 7800 11950 7800
+Wire Wire Line
+	11950 7800 11950 6200
+Wire Wire Line
+	11950 6200 23200 6200
+Wire Wire Line
+	12700 7900 12450 7900
+Wire Wire Line
+	12450 7900 12450 7150
+Connection ~ 22150 7700
+Wire Wire Line
+	22150 7700 22150 7800
+Wire Wire Line
+	22150 7800 22200 7800
+Wire Wire Line
+	23000 7700 23000 7650
+Wire Wire Line
+	23000 7650 21700 7650
+Wire Wire Line
+	21700 7650 21700 7350
+Wire Wire Line
+	23000 7900 23000 7850
+Wire Wire Line
+	23000 7850 22000 7850
+Wire Wire Line
+	22000 7850 22000 7550
+Wire Wire Line
+	23000 8000 23000 8050
+Wire Wire Line
+	23000 8050 21900 8050
+Wire Wire Line
+	21900 8050 21900 7750
+Wire Wire Line
+	23000 8100 23000 8150
+Wire Wire Line
+	23000 8150 12550 8150
+Wire Wire Line
+	23000 7400 23150 7400
+Wire Wire Line
+	23150 7400 23150 6050
+Wire Wire Line
+	23000 7300 23100 7300
+Wire Wire Line
+	23100 7300 23100 5900
 Connection ~ 23400 8800
 Wire Wire Line
@@
 	23450 10850 12100 10850
 Wire Wire Line
-	12100 10850 12100 7600
-Wire Wire Line
-	12100 7600 12700 7600
-Wire Wire Line
 	23000 7600 23300 7600
 Wire Wire Line
@@
 Wire Wire Line
 	14200 7050 14500 7050
-Wire Wire Line
-	13500 7500 13500 6050
-Wire Wire Line
-	13500 6050 23000 6050
-Wire Wire Line
-	23000 6050 23000 7300
 Connection ~ 20500 6950
 Wire Wire Line
@@
 Connection ~ 20500 7250
 Wire Wire Line
-	23000 7700 23400 7700
-Wire Wire Line
-	23400 7700 23400 7250
-Wire Wire Line
-	23400 7250 14500 7250
+	14500 7250 23400 7250
 Connection ~ 20500 7450
 Wire Wire Line
-	23000 7800 23450 7800
-Wire Wire Line
-	23450 7800 23450 7450
-Wire Wire Line
-	23450 7450 13650 7450
+	13650 7450 23450 7450
 Connection ~ 20500 7750
-Wire Wire Line
-	22200 7900 21900 7900
-Wire Wire Line
-	21900 7900 21900 7750
 Wire Wire Line
 	21900 7750 12650 7750
 Connection ~ 20500 8150
-Wire Wire Line
-	22200 8100 22200 8150
-Wire Wire Line
-	22200 8150 12550 8150
 Connection ~ 20500 8350
 Wire Wire Line
@@
 Connection ~ 7000 10050
 Connection ~ 14500 7150
-Wire Wire Line
-	12700 7800 12450 7800
-Wire Wire Line
-	12450 7800 12450 7150
 Connection ~ 14500 7550
 Wire Wire Line
@@
 	13650 8000 13500 8000
 Connection ~ 14500 7450
-Wire Wire Line
-	12350 6950 12350 7700
-Wire Wire Line
-	12350 7700 12700 7700
 Connection ~ 14500 6950
 Connection ~ 7000 9650
@@
 	23100 8200 23000 8200
 Connection ~ 20500 8250
-Wire Wire Line
-	12600 7950 22200 7950
-Wire Wire Line
-	22200 7950 22200 8000
 Connection ~ 20500 7950
 Wire Wire Line
 	12550 7550 22000 7550
-Wire Wire Line
-	22000 7550 22000 7800
-Wire Wire Line
-	22000 7800 22200 7800
 Connection ~ 20500 7550
 Wire Wire Line
-	14500 7350 21700 7350
-Wire Wire Line
-	21700 7350 21700 7700
-Wire Wire Line
-	21700 7700 22200 7700
+	21700 7350 14500 7350
 Connection ~ 20500 7350
 Wire Wire Line
@@
 Connection ~ 20500 7150
 Wire Wire Line
-	12700 7500 12700 5900
-Wire Wire Line
-	12700 5900 22200 5900
-Wire Wire Line
-	22200 5900 22200 7300
-Wire Wire Line
-	13500 7600 13600 7600
-Wire Wire Line
-	13600 7600 13600 6200
-Wire Wire Line
-	13600 6200 23200 6200
-Wire Wire Line
-	23200 6200 23200 7400
-Wire Wire Line
-	23200 7400 23000 7400
-Wire Wire Line
 	20500 9350 23400 9350
 Wire Wire Line
 	23400 9350 23400 8800
+Wire Wire Line
+	22200 7300 22200 6700
+Wire Wire Line
+	22200 6700 21750 6700
+Wire Wire Line
+	22200 7400 22150 7400
+Wire Wire Line
+	22150 7400 22150 6700
+Connection ~ 22150 6700
+Wire Wire Line
+	23200 6200 23200 7500
+Wire Wire Line
+	23200 7500 23000 7500
+Wire Wire Line
+	12600 7950 21700 7950
+Wire Wire Line
+	21700 7950 21700 8100
+Wire Wire Line
+	21700 8100 22200 8100
+Wire Wire Line
+	23450 7450 23450 7950
+Wire Wire Line
+	23450 7950 22200 7950
+Wire Wire Line
+	22200 7950 22200 8000
+Wire Wire Line
+	23400 7250 23400 7800
+Wire Wire Line
+	23400 7800 23000 7800
+Wire Wire Line
+	22200 7700 22050 7700
+Wire Wire Line
+	22050 7700 22050 6700
+Connection ~ 22050 6700
+Wire Wire Line
+	22200 7900 22100 7900
+Wire Wire Line
+	22100 7900 22100 7700
+Connection ~ 22100 7700
+Wire Wire Line
+	12350 6950 12350 7850
+Wire Wire Line
+	12350 7850 13500 7850
+Wire Wire Line
+	13500 7850 13500 7800
+Wire Wire Line
+	13500 7700 13500 7650
+Wire Wire Line
+	13500 7650 12100 7650
+Wire Wire Line
+	12100 7650 12100 10850
+Wire Wire Line
+	13550 6050 13550 7600
+Wire Wire Line
+	13550 7600 13500 7600
+Wire Wire Line
+	13450 5900 13450 7500
+Wire Wire Line
+	13450 7500 13500 7500
+Wire Wire Line
+	12700 7600 12650 7600
+Wire Wire Line
+	12650 7600 12650 6450
+Connection ~ 12650 6450
+Text Label 12300 6450 0    60   ~ 0
+GND
+$Comp
+L CONN_20X2 Linker?
+U 1 1 503360E8
+P 13100 8450
+F 0 "Linker?" H 13100 9500 60  0000 C CNN
+F 1 "CONN_20X2" V 13100 8450 50  0000 C CNN
+	1    13100 8450
+	1    0    0    -1
+$EndComp
+Text Label 21950 6700 0    60   ~ 0
+GND
+$Comp
+L CONN_20X2 LinkerToTB?
+U 1 1 50335E74
+P 22600 8250
+F 0 "LinkerToTB?" H 22600 9300 60  0000 C CNN
+F 1 "CONN_20X2" V 22600 8250 50  0000 C CNN
+	1    22600 8250
+	1    0    0    -1
+$EndComp
+NoConn ~ 9700 9300
+NoConn ~ 23000 9200
+NoConn ~ 23000 9100
+NoConn ~ 22200 9100
+NoConn ~ 22200 8900
+NoConn ~ 22200 8700
+NoConn ~ 23000 8500
 Text Label 21150 9350 0    60   ~ 0
 RBI
@@
 NoConn ~ 9700 7800
 NoConn ~ 9700 7700
-NoConn ~ 12700 7900
 NoConn ~ 12700 8900
 NoConn ~ 12700 9100
@@
 NoConn ~ 13500 8100
 NoConn ~ 13500 7900
-NoConn ~ 13500 7800
-NoConn ~ 13500 7700
 NoConn ~ 14500 7650
 NoConn ~ 14500 7850
@@
 Text Label 13800 6050 0    60   ~ 0
 -AIN2
-Text Label 12950 5900 0    60   ~ 0
+Text Label 13700 5900 0    60   ~ 0
 +AIN2
 Text Label 4500 6000 0    60   ~ 0
@@
 L CONN_20X2 LinkerToTB1
 U 1 1 4FB20BA1
-P 22600 8250
-F 0 "LinkerToTB1" H 22600 9300 60  0000 C CNN
-F 1 "CONN_20X2" V 22600 8250 50  0000 C CNN
-	1    22600 8250
+P 25800 8400
+F 0 "LinkerToTB1" H 25800 9450 60  0000 C CNN
+F 1 "CONN_20X2" V 25800 8400 50  0000 C CNN
+	1    25800 8400
 	1    0    0    1
 $EndComp
@@
 L CONN_20X2 Linker1
 U 1 1 4FB209DE
-P 13100 8450
-F 0 "Linker1" H 13100 9500 60  0000 C CNN
-F 1 "CONN_20X2" V 13100 8450 50  0000 C CNN
-	1    13100 8450
+P 25800 11250
+F 0 "Linker1" H 25800 12300 60  0000 C CNN
+F 1 "CONN_20X2" V 25800 11250 50  0000 C CNN
+	1    25800 11250
 	1    0    0    1
 $EndComp
@@
 L CONN_20X2 Linker2
 U 1 1 4FB209CD
-P 9300 8450
-F 0 "Linker2" H 9300 9500 60  0000 C CNN
-F 1 "CONN_20X2" V 9300 8450 50  0000 C CNN
-	1    9300 8450
+P 9650 10750
+F 0 "Linker2" H 9650 11800 60  0000 C CNN
+F 1 "CONN_20X2" V 9650 10750 50  0000 C CNN
+	1    9650 10750
 	1    0    0    1
 $EndComp
