File: adapterboardV2.sch (KiCad schematic (older format))
At the start: 43 parts, among them P1 CONN_2, P2 CONN_2, P3 CONN_2, P4 CONN_2, P5 CONN_2

Commit message: Forced to take newer files, disregarding any merge conflicts
Parts:
- added K1, K2, K3, K4: Vext/+5_ANA, symbol CONN_3
- added P10: RBI, symbol CONN_2
- added P11: CS, symbol CONN_2
- added P12: R12, symbol CONN_2
- added P13: SR, symbol CONN_2
- added P14: IS1, symbol CONN_2
- added P15: RESET, symbol CONN_2
- added P16: SPHI1, symbol CONN_2
- added P17: SPHI2, symbol CONN_2
- added P18: SBI, symbol CONN_2
- added P19: SEB, symbol CONN_2
- added P20: LE, symbol CONN_2
- added P21, P22, P23, P24: GND, symbol CONN_2
- added P25: +AIN1, symbol CONN_2
- added P26: -AIN1, symbol CONN_2
- added P27: +AIN2, symbol CONN_2
- added P28: -AIN2, symbol CONN_2
- added P29, P30, P6: CONN_1, symbol CONN_1
- added P7: IS2, symbol CONN_2
- added P8: RPHI1, symbol CONN_2
- added P9: RPHI2, symbol CONN_2
- added R12Switch1, SRSwitch1: SWITCH_INV_MSM, symbol SWITCH_INV_MSM
- added R27: 100ohm, symbol R
- added R28: 300ohm, symbol R
- added R29, R30, R31, R32, R33, R34, R35, R36: R, ~, symbol R
- added Sequencer1, Telescope_2: CONN_20X2, symbol CONN_20X2
- P1: value CONN_2 -> GND
- P2: value CONN_2 -> CAL
- P3: value CONN_2 -> AREF
- P4: value CONN_2 -> Vthr
- P5: value CONN_2 -> RG
- renumbered Telescope1 to Telescope_1
Connections:
- net labels added: IS2, R12_VD, SR_VD, VTransto+1, VTransto+2, VTransto-1, VTransto-2, Vext
- wire segments 138 -> 285
- no-connect marks 34 -> 45
Other:
- moved on the sheet: HVin1, Null1, NullCap1, P1, Telescope_1, Testboard1, Testboard2
