File: SensorBoard2013.sch (KiCad schematic (older format))
At the start: 16 parts, among them P1 CONN_20X2, P2 CONN_20X2, P3 CONN_1

Commit message: Latest file from Tilman
Parts:
- gave numbers to parts that had none: 1
Changed lines of the file:
@@
-EESchema Schematic File Version 2  date Mon Aug 26 10:59:18 2013
+EESchema Schematic File Version 2  date Mon Aug 26 11:00:25 2013
 LIBS:power
 LIBS:device
@@
 Aref
 $Comp
-L R R?
+L R R1
 U 1 1 521B188A
 P 6050 4950
-F 0 "R?" V 6130 4950 50  0000 C CNN
+F 0 "R1" V 6130 4950 50  0000 C CNN
 F 1 "R" V 6050 4950 50  0000 C CNN
 	1    6050 4950
