File: motherboard2015/motherboard2015.sch (KiCad schematic (older format))
At the start: 27 parts

Commit message: Updates to motherboard2015
Parts:
- added RP1, RP2: R_PACK8, extras:R8_MNR18, symbol R_PACK8
- C1, C10, C11, C12, C13, C14, C2, C3, C4, C5, C6, C7, C8, C9: renamed from C?; footprint (none) -> SMD_Packages:SMD-0603
- J1, J2, J3, J4: renamed from J?; footprint (none) -> Connect:RJ45_8
- MEC1, MEC2, MEC3, MEC4: renamed from MEC?; footprint (none) -> extras:MEC1
- P1: renamed from P?; footprint (none) -> Pin_Headers:Pin_Header_Straight_2x20
- RP3, RP4, RP5, RP6: renamed from RP?; value 100R -> 90R; footprint (none) -> extras:R8_MNR18
Connections:
- net CAL: now also RP1.5 (P5)
- net CS: now also RP2.2 (P2)
- net GND: now also RP1.10 (R7), RP1.11 (R6), RP1.12 (R5), RP1.13 (R4), RP1.14 (R3), RP1.15 (R2), RP1.16 (R1), RP1.9 (R8), RP2.10 (R7), RP2.11 (R6), RP2.12 (R5), RP2.13 (R4), RP2.14 (R3), RP2.15 (R2), RP2.16 (R1), RP2.9 (R8)
- net IS1: now also RP2.6 (P6)
- net IS2: now also RP2.5 (P5)
- net LE: now also RP2.8 (P8)
- net R12: now also RP2.3 (P3)
- net RBI: now also RP2.1 (P1)
- net RPHI1: now also RP1.7 (P7)
- net RPHI2: now also RP1.6 (P6)
- net Reset: now also RP2.7 (P7)
- net SBI: now also RP1.3 (P3)
- net SEB: now also RP1.4 (P4)
- net SPHI1: now also RP1.2 (P2)
- net SPHI2: now also RP1.1 (P1)
- net SR: now also RP2.4 (P4)
Other:
- note added: "Terminal\nResistors\n(optional)"
- moved on the sheet: P1
