File: APC128testboard/APC128testboard_ampstage.sch (KiCad schematic (older format))
At the start: 23 parts, among them U2 ADA4950-1, U6 AD8130, U7 AD8130

Commit message: Final touchups for APC128testboard submission.
Parts:
- added R14, R15: 0, symbol R
Connections:
- wire segments 63 -> 71
- no-connect marks 2 -> 0
Other:
- note added: "connect 0 Ohm resistors \nfor x3 amplification"
Changed lines of the file:
@@
 Text Label 2900 2150 0    60   ~ 0
 GND
-Text Label 3600 2000 0    60   ~ 0
+Text Label 2950 1900 0    60   ~ 0
 IN+
-Text Label 3600 2300 0    60   ~ 0
+Text Label 2950 2400 0    60   ~ 0
 IN-
 Text Label 7100 4100 0    60   ~ 0
@@
 Text Label 7100 3450 0    60   ~ 0
 4950OUT+
-NoConn ~ 3850 2100
-NoConn ~ 3850 2200
 $Comp
 L C C2
@@
 Connection ~ 3150 2150
 Wire Wire Line
-	3850 2000 3600 2000
-Wire Wire Line
-	3850 2300 3600 2300
+	3850 1900 3850 2000
+Wire Wire Line
+	3850 2400 3850 2300
 Wire Wire Line
 	2700 5200 3550 5200
@@
 Connection ~ 2700 4400
 Wire Wire Line
-	3550 3600 2700 3600
+	2700 3600 3550 3600
 Connection ~ 3450 1800
 Connection ~ 3250 2900
@@
 	4550 5650 4600 5650
 Connection ~ 4550 5450
+$Comp
+L R R14
+U 1 1 53A1CCE6
+P 3550 2050
+F 0 "R14" V 3630 2050 40  0000 C CNN
+F 1 "0" V 3557 2051 40  0000 C CNN
+F 2 "" V 3480 2050 30  0000 C CNN
+F 3 "" H 3550 2050 30  0000 C CNN
+	1    3550 2050
+	0    1    1    0
+$EndComp
+$Comp
+L R R15
+U 1 1 53A1CD33
+P 3550 2250
+F 0 "R15" V 3630 2250 40  0000 C CNN
+F 1 "0" V 3557 2251 40  0000 C CNN
+F 2 "" V 3480 2250 30  0000 C CNN
+F 3 "" H 3550 2250 30  0000 C CNN
+	1    3550 2250
+	0    1    1    0
+$EndComp
+Wire Wire Line
+	2950 2400 3850 2400
+Wire Wire Line
+	3300 2400 3300 2250
+Wire Wire Line
+	2950 1900 3850 1900
+Wire Wire Line
+	3300 1900 3300 2050
+Connection ~ 3300 1900
+Connection ~ 3300 2400
+Wire Wire Line
+	3800 2250 3800 2200
+Wire Wire Line
+	3800 2200 3850 2200
+Wire Wire Line
+	3800 2050 3800 2100
+Wire Wire Line
+	3800 2100 3850 2100
+Text Notes 2800 2600 1    60   ~ 0
+connect 0 Ohm resistors \nfor x3 amplification
 $EndSCHEMATC

Commit message: Updated some passive values based on what is actually on the board.
Parts:
- C16, C17: value C -> NC
- R2, R3: value R -> NC
- R4, R5: value R -> 0
Changed lines of the file:
@@
 P 4800 5450
 F 0 "R5" V 4880 5450 40  0000 C CNN
-F 1 "R" V 4807 5451 40  0000 C CNN
+F 1 "0" V 4807 5451 40  0000 C CNN
 F 2 "" V 4730 5450 30  0000 C CNN
 F 3 "" H 4800 5450 30  0000 C CNN
@@
 P 4000 5450
 F 0 "R3" V 4080 5450 40  0000 C CNN
-F 1 "R" V 4007 5451 40  0000 C CNN
+F 1 "NC" V 4007 5451 40  0000 C CNN
 F 2 "" V 3930 5450 30  0000 C CNN
 F 3 "" H 4000 5450 30  0000 C CNN
@@
 P 4800 3350
 F 0 "R4" V 4880 3350 40  0000 C CNN
-F 1 "R" V 4807 3351 40  0000 C CNN
+F 1 "0" V 4807 3351 40  0000 C CNN
 F 2 "" V 4730 3350 30  0000 C CNN
 F 3 "" H 4800 3350 30  0000 C CNN
@@
 P 4000 3350
 F 0 "R2" V 4080 3350 40  0000 C CNN
-F 1 "R" V 4007 3351 40  0000 C CNN
+F 1 "NC" V 4007 3351 40  0000 C CNN
 F 2 "" V 3930 3350 30  0000 C CNN
 F 3 "" H 4000 3350 30  0000 C CNN
@@
 P 4800 5650
 F 0 "C17" H 4800 5750 40  0000 L CNN
-F 1 "C" H 4806 5565 40  0000 L CNN
+F 1 "NC" H 4806 5565 40  0000 L CNN
 F 2 "" H 4838 5500 30  0000 C CNN
 F 3 "" H 4800 5650 60  0000 C CNN
@@
 P 4800 3150
 F 0 "C16" H 4800 3250 40  0000 L CNN
-F 1 "C" H 4806 3065 40  0000 L CNN
+F 1 "NC" H 4806 3065 40  0000 L CNN
 F 2 "" H 4838 3000 30  0000 C CNN
 F 3 "" H 4800 3150 60  0000 C CNN

Commit message: fixes broken passives in APC128 testboard schematic
Connections:
- wire segments 71 -> 89
Changed lines of the file:
@@
 LIBS:conn-scsi68
 LIBS:APC128testboard-cache
-EELAYER 24 0
+EELAYER 25 0
 EELAYER END
 $Descr A4 11693 8268
@@
 	2800 5000 3550 5000
 Wire Wire Line
-	3250 5000 3250 4800
-Wire Wire Line
-	3050 5000 3050 4800
+	3250 4750 3250 5000
+Wire Wire Line
+	3050 4750 3050 5000
 Connection ~ 3250 5000
 Wire Wire Line
 	4450 5000 5250 5000
 Wire Wire Line
-	4750 5000 4750 4800
-Wire Wire Line
-	4950 5000 4950 4800
+	4750 4750 4750 5000
+Wire Wire Line
+	4950 4750 4950 5000
 Connection ~ 4750 5000
 Wire Wire Line
-	3250 3800 3250 4000
+	3250 3800 3250 4050
 Wire Wire Line
 	2800 3800 3550 3800
 Wire Wire Line
-	3050 4000 3050 3800
+	3050 3800 3050 4050
 Connection ~ 3250 3800
 Wire Wire Line
-	4750 4000 4750 3800
+	4750 3800 4750 4050
 Wire Wire Line
 	4450 3800 5250 3800
 Wire Wire Line
-	4950 3800 4950 4000
+	4950 3800 4950 4050
 Connection ~ 4750 3800
 Wire Wire Line
@@
 Connection ~ 3250 1400
 Wire Wire Line
-	5050 5100 5050 5650
+	5050 5650 5050 5100
 Connection ~ 5050 5100
 Wire Wire Line
@@
 	4550 5200 4450 5200
 Wire Wire Line
-	4550 5450 4250 5450
-Wire Wire Line
-	3750 5450 3450 5450
+	4150 5450 4650 5450
+Wire Wire Line
+	3450 5450 3850 5450
 Wire Wire Line
 	3450 5450 3450 5200
@@
 	4550 3600 4450 3600
 Wire Wire Line
-	4550 3350 4250 3350
-Wire Wire Line
-	3750 3350 3450 3350
+	4150 3350 4650 3350
+Wire Wire Line
+	3450 3350 3850 3350
 Wire Wire Line
 	3450 3350 3450 3600
 Connection ~ 3450 3600
 Wire Wire Line
-	5050 3150 5000 3150
+	4950 3150 5050 3150
 Connection ~ 5050 3350
 Wire Wire Line
-	4600 3150 4550 3150
+	4550 3150 4650 3150
 Connection ~ 4550 3350
 Wire Wire Line
-	5050 5650 5000 5650
+	4950 5650 5050 5650
 Connection ~ 5050 5450
 Wire Wire Line
-	4550 5650 4600 5650
+	4550 5650 4650 5650
 Connection ~ 4550 5450
 $Comp
@@
 Text Notes 2800 2600 1    60   ~ 0
 connect 0 Ohm resistors \nfor x3 amplification
+Wire Wire Line
+	3250 4350 3250 4450
+Wire Wire Line
+	3050 4350 3050 4450
+Wire Wire Line
+	4950 3350 5050 3350
+Wire Wire Line
+	4950 4350 4950 4450
+Wire Wire Line
+	4750 4350 4750 4450
+Wire Wire Line
+	4950 5450 5050 5450
+Wire Wire Line
+	3450 2900 3450 2850
+Wire Wire Line
+	3250 2900 3250 2850
+Wire Wire Line
+	3250 2550 3250 2500
+Wire Wire Line
+	3450 2500 3450 2550
+Wire Wire Line
+	3300 2250 3400 2250
+Wire Wire Line
+	3800 2250 3700 2250
+Wire Wire Line
+	3800 2050 3700 2050
+Wire Wire Line
+	3300 2050 3400 2050
+Wire Wire Line
+	3450 1800 3450 1750
+Wire Wire Line
+	3250 1800 3250 1750
+Wire Wire Line
+	3250 1400 3250 1450
+Wire Wire Line
+	3450 1400 3450 1450
 $EndSCHEMATC
