File: DAQCard2015/ADCChannel2.sch (KiCad schematic (older format))
At the start: 21 parts, among them U4 THS4524IDBTR, U5 AD9219

Commit message: propogate previous changes to other channels and schematic
Parts:
- removed C11: 10uF, Capacitors_SMD:C_0805, symbol CP
- removed C12, C14, C15, C16, C18, C19: .1uF, Capacitors_SMD:C_0603, symbol C
- removed C13: 10000pF, Capacitors_SMD:C_0603, symbol C
- removed C17: 2.2uF, Capacitors_SMD:C_0805, symbol CP
- removed R11, R12, R13, R14: Rt, Resistors_SMD:R_0603, symbol R
- removed R15: 2.7k, Resistors_SMD:R_0603, symbol R
- removed R16: 1k, Resistors_SMD:R_0603, symbol R
- removed R17: 10k, Resistors_SMD:R_0603, symbol R
- removed RP4: Ri, extras:R8_MNR18, symbol R_PACK8
- removed RP5, RP6: Rf, extras:R4-MNR04, symbol R_PACK4
- removed U4: THS4524IDBTR, Housings_SSOP:TSSOP-38_4.4x9.7mm_Pitch0.5mm, symbol THS4524IDBTR
- removed U5: AD9219, SMD_Packages:QFN-48-1EP, symbol AD9219
- added C47, C48, C49, C51, C52: .1uF, Capacitors_SMD:C_0603, symbol C
- added C50: 2.2uF, Capacitors_SMD:C_0805, symbol C
- added R41, R42, R43, R44: Rt, Resistors_SMD:R_0603, symbol R
- added R45: 10k, Resistors_SMD:R_0603, symbol R
- added RP22: Ri, extras:R8_MNR18, symbol R_PACK8
- added RP23, RP24: Rf, extras:R4-MNR04, symbol R_PACK4
- added U17: THS4524IDBTR, Housings_SSOP:TSSOP-38_4.4x9.7mm_Pitch0.5mm, symbol THS4524IDBTR
- added U18: AD9219, extras:QFN-48-1EP, symbol AD9219
Connections:
- net 1V8ana: now also U18.1 (AVDD), U18.10 (AVDD), U18.2 (AVDD), U18.27 (AVDD), U18.32 (AVDD), U18.35 (AVDD), U18.36 (AVDD), U18.39 (AVDD), U18.41 (SENSE), U18.45 (AVDD), U18.46 (AVDD), U18.5 (AVDD), U18.6 (AVDD), U18.9 (AVDD)
- net 1V8dig: now also U18.12 (DRVDD), U18.25 (DRVDD)
- net 3V3ana: now also U17.20 (VS4+), U17.25 (VS3+), U17.30 (VS2+), U17.35 (VS1+)
- net ADC_CLK+: now also C48.2
- net ADC_CLK-: now also C47.2
- net ADC_CSB: now also U18.30 (CSB)
- net ADC_SCLK: now also U18.28 (SCLK/DTP)
- net ADC_SDIO: now also U18.29 (SDIO/ODM)
- net ADC_Vref: now also U18.42 (VREF)
- net CHA+: now also RP24.6 (R3), U17.36 (VOUT1+), U18.33 (VIN+A)
- net CHA-: now also RP24.5 (R4), U17.37 (VOUT1-), U18.34 (VIN-A)
- net CHB+: now also RP24.8 (R1), U17.31 (VOUT2+), U18.38 (VIN+B)
- net CHB-: now also RP24.7 (R2), U17.32 (VOUT2-), U18.37 (VIN-B)
- net CHC+: now also RP23.6 (R3), U17.26 (VOUT3+), U18.47 (VIN+C)
- net CHC-: now also RP23.5 (R4), U17.27 (VOUT3-), U18.48 (VIN-C)
- net CHD+: now also RP23.8 (R1), U17.21 (VOUT4+), U18.4 (VIN+D)
- net CHD-: now also RP23.7 (R2), U17.22 (VOUT4-), U18.3 (VIN-D)
- net D+A: now also U18.20 (D+A)
- net D+B: now also U18.18 (D+B)
- net D+C: now also U18.16 (D+C)
- net D+D: now also U18.14 (D+D)
- net D-A: now also U18.19 (D-A)
- net D-B: now also U18.17 (D-B)
- net D-C: now also U18.15 (D-C)
- net D-D: now also U18.13 (D-D)
- net DCO+: now also U18.24 (DCO+)
- net DCO-: now also U18.23 (DCO-)
- net EXT_CHA+: now also R41.1, RP22.1 (P1)
- net EXT_CHA-: now also R41.2, RP22.2 (P2)
- net EXT_CHB+: now also R42.1, RP22.3 (P3)
- net EXT_CHB-: now also R42.2, RP22.4 (P4)
- net EXT_CHC+: now also R43.1, RP22.5 (P5)
- net EXT_CHC-: now also R43.2, RP22.6 (P6)
- net EXT_CHD+: now also R44.1, RP22.7 (P7)
- net EXT_CHD-: now also R44.2, RP22.8 (P8)
- net FCO+: now also U18.22 (FCO+)
- net FCO-: now also U18.21 (FCO-)
- new net: RP22.12 (R5), RP23.1 (P1), U17.12 (VIN3+)
- new net: RP22.11 (R6), RP23.2 (P2), U17.13 (VIN3-)
- new net: RP22.10 (R7), RP23.3 (P3), U17.17 (VIN4+)
- new net: RP22.9 (R8), RP23.4 (P4), U17.18 (VIN4-)
- new net: RP22.16 (R1), RP24.1 (P1), U17.2 (Vin1+)
- new net: RP22.15 (R2), RP24.2 (P2), U17.3 (VIN1-)
- new net: RP22.14 (R3), RP24.3 (P3), U17.7 (VIN2+)
- new net: RP22.13 (R4), RP24.4 (P4), U17.8 (VIN2-)
- new net: C48.1, U18.8 (CLK+)
- new net: R45.2, U18.40 (RBIAS)
- new net: C50.2, C51.1, C52.2, U18.43 (REFB)
- new net: C49.1, C50.1, C51.2, U18.44 (REFT)
- new net: C47.1, U18.7 (CLK-)
- new net GND: C49.2, C52.1, R45.1, U17.10 (VS-), U17.15 (VS-), U17.23 (VS-), U17.24 (VS-), U17.28 (VS-), U17.29 (VS-), U17.33 (VS-), U17.34 (VS-), U17.38 (VS-), U17.5 (VS-), U18.0 (AGND), U18.11 (DRGND), U18.26 (DRGND), U18.31 (PDWN)
- new net Vocm: U17.14 (VOCM3), U17.19 (VOCM4), U17.4 (VOCM1), U17.9 (VOCM2)
Other:
- note added: "PD floating -> Power On"
- note removed: "0.9V"
