File: DAQCard2015/DAQCard2015.kicad_pcb (KiCad board)
At the start: 2 copper layers, 207 parts, among them CON1 BARREL_JACK, P1 QTH-090-01-F-D-A, P2 QTH-090-01-F-D-A, P3 miniDIL20, P4 LEMO_EPY.00.250.NTN, P5 LEMO_EPY.00.250.NTN, U1 AD5628, U10 THS4524IDBTR, U11 AD9219, U12 THS4524IDBTR, U13 AD9219, U14 THS4524IDBTR, U15 AD9219, U16 THS4524IDBTR, U17 AD9219, U18 APXS002A0X-SRZ, U19 APXS002A0X-SRZ, U2 THS4524IDBTR, U20 APXS002A0X-SRZ, U21 MCP1826, U22 RJ45x8, U3 AD9219, U4 THS4524IDBTR, U5 AD9219, U6 THS4524IDBTR, U7 AD9219, U8 THS4524IDBTR, U9 AD9219

Commit message: Updates to DAQCard2015, especially to power systems
Parts:
- C13, C22, C31, C4, C40, C49, C58, C67: value .01uF -> 10000pF
- C80, C81: value 10nF -> 10000pF
- RP1: value RP8 -> Ri
- RP10, RP13, RP16, RP19, RP22, RP4, RP7: value R_PACK8 -> Ri
- U3: footprint SMD_Packages:QFN-48-1EP -> extras:QFN-48-1EP
- moved C89 102.6 mm to (46.5, 67.5), turned to 180 degrees
- moved U1 86.1 mm to (136.4, 41.6)
- moved RP4 79.8 mm to (196.0, 22.6)
- moved U5 79.8 mm to (198.0, 43.0)
- moved R13 79.8 mm to (193.8, 22.2)
- moved RP18 79.8 mm to (209.8, 31.0)
- moved RP5 79.8 mm to (197.4, 34.2)
- moved RP6 79.8 mm to (200.8, 34.2)
- moved U4 79.8 mm to (197.2, 28.2)
- moved RP2 79.4 mm to (148.0, 40.5)
- moved U3 78.7 mm to (154.7, 50.0)
- moved R18 78.7 mm to (257.6, 23.1)
- moved R19 78.7 mm to (261.6, 17.5)
- moved R48 78.7 mm to (277.6, 27.1)
- moved RP20 78.7 mm to (279.6, 35.3)
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Connections:
- RP2 pad 1: Net-(RP1-Pad10) -> Net-(RP1-Pad12)
- RP2 pad 2: Net-(RP1-Pad9) -> Net-(RP1-Pad11)
- RP2 pad 3: Net-(RP1-Pad12) -> Net-(RP1-Pad10)
- RP2 pad 4: Net-(RP1-Pad11) -> Net-(RP1-Pad9)
- RP3 pad 1: Net-(RP1-Pad14) -> Net-(RP1-Pad16)
- RP3 pad 2: Net-(RP1-Pad13) -> Net-(RP1-Pad15)
- RP3 pad 3: Net-(RP1-Pad16) -> Net-(RP1-Pad14)
- RP3 pad 4: Net-(RP1-Pad15) -> Net-(RP1-Pad13)
- U1 pad 15: /Frontend/ADC_CLK- -> /Frontend/ADC_SDIO
- U1 pad 16: /Frontend/ADC_CLK+ -> /Frontend/ADC_SCLK
- U22 pad 4: /Frontend/ADCChannel1/EXT_CHC+ -> /Frontend/ADCChannel1/EXT_CHB-
- U22 pad 5: /Frontend/ADCChannel1/EXT_CHB- -> /Frontend/ADCChannel1/EXT_CHB+
- U22 pad 6: /Frontend/ADCChannel1/EXT_CHB+ -> /Frontend/ADCChannel1/EXT_CHC+
Routing:
- net /Frontend/ADCChannel1/EXT_CHD-: track 0.00 -> 26.1 mm
- net /Frontend/ADCChannel1/EXT_CHC-: track 0.00 -> 23.4 mm
- net /Frontend/ADCChannel1/EXT_CHD+: track 0.00 -> 22.9 mm
- net /Frontend/ADCChannel1/EXT_CHC+: track 0.00 -> 22.5 mm, vias 0 -> 2
- net /Frontend/ADCChannel1/EXT_CHA-: track 0.00 -> 21.9 mm
- net /Frontend/ADCChannel1/EXT_CHB+: track 0.00 -> 21.2 mm
- net /Frontend/ADCChannel1/EXT_CHA+: track 0.00 -> 20.3 mm
- net /Frontend/ADCChannel1/EXT_CHB-: track 0.00 -> 19.4 mm
- net Net-(C10-Pad2): track 0.00 -> 18.4 mm, vias 0 -> 2
- net Net-(C7-Pad1): track 0.00 -> 17.1 mm, vias 0 -> 2
- net /Frontend/ADCChannel1/CHA+: track 0.00 -> 13.8 mm, vias 0 -> 2
- net /Frontend/ADCChannel1/CHB+: track 0.00 -> 13.5 mm
- net Net-(RP1-Pad9): track 0.00 -> 13.4 mm, vias 0 -> 2
- net Net-(RP1-Pad10): track 0.00 -> 13.2 mm, vias 0 -> 2
- net Net-(RP1-Pad11): track 0.00 -> 13.2 mm, vias 0 -> 2
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Other:
- copper layers 2 -> 4
- net class Default: clearance 0.2 -> 0.127; trace_width 0.25 -> 0.508; via_dia 0.6 -> 0.4572; via_drill 0.4 -> 0.3048
- rule trace_clearance: 0.2 -> 0.127
- rule trace_min: 0.2 -> 0.1524
- rule via_min_drill: 0.3 -> 0.0254
- rule via_min_size: 0.4 -> 0.0381

Commit message: propogate previous changes to other channels and schematic
Parts:
- removed the C4 at (111.0, 107.2)
- removed the C53 at (115.6, 133.4)
- removed the C56 at (108.0, 135.0)
- removed the C57 at (129.2, 94.0)
- removed the C58 at (116.0, 97.2)
- removed the C62 at (108.0, 142.4)
- removed the C63 at (169.6, 129.0)
- removed the C64 at (168.8, 97.4)
- removed the C65 at (115.6, 141.6)
- removed the C66 at (100.8, 142.4)
- removed the C67 at (96.6, 143.2)
- removed the C68 at (124.2, 140.8)
- removed the C69 at (164.4, 136.2)
- removed C70, C72, C73: .1uF, Capacitors_SMD:C_0603
- removed C71: 2.2uF, extras:SMD_Cap_3mmDia
- removed C77, C78, C79, C89: 10uF, extras:SMD_Cap_3mmDia
- removed the R4 at (160.0, 27.7)
- removed the R46 at (275.0, 19.9)
- removed the R47 at (285.4, 23.7)
- removed the R48 at (277.6, 27.1)
- removed the R49 at (272.2, 28.9)
- removed the R5 at (157.0, 27.7)
- removed the R50 at (124.8, 149.0)
- removed the R51 at (176.4, 142.2)
- removed R53, R54, R55, R56: Rt, Resistors_SMD:R_0603
- removed R57: 2.7k, Resistors_SMD:R_0603
- removed R58: 1k, Resistors_SMD:R_0603
- removed R59: 10k, Resistors_SMD:R_0603
- removed the U2 at (155.0, 40.5)
- removed the U21 at (64.6, 93.4)
- added C1: 10uF, Capacitors_SMD:C_0805, F.Cu at (6.50, -20.5)
- added D1: LED, LEDs:LED-1206, F.Cu at (-32.0, 29.0)
- added R1: 2.7k, Resistors_SMD:R_0603, F.Cu at (-40.5, 32.5)
- added R2: 1k, Resistors_SMD:R_0603, F.Cu at (-24.5, 9.50)
- added SW1: SPST, extras:Switch_ES02MSABE, F.Cu at (19.4, 48.9)
- added U18: AD9219, extras:QFN-48-1EP, F.Cu at (195.5, 31.8)
- added U19: CDBHD240-G, extras:mini-DIP4, F.Cu at (17.2, 65.2)
- added U20: LM1086, extras:TO-263-4, F.Cu at (29.2, 50.5)
- C11, C2, C29, C47: value 10uF -> .1uF; footprint extras:SMD_Cap_3mmDia -> Capacitors_SMD:C_0603
- C13, C22, C31, C40, C49: value 10000pF -> .1uF
- C14, C32, C50: value .1uF -> 2.2uF; footprint Capacitors_SMD:C_0603 -> Capacitors_SMD:C_0805
- C17, C35: value 2.2uF -> .1uF; footprint extras:SMD_Cap_3mmDia -> Capacitors_SMD:C_0603
- C20, C38: value 10uF -> 2.2uF; footprint extras:SMD_Cap_3mmDia -> Capacitors_SMD:C_0805
- C26, C44, C8: footprint extras:SMD_Cap_3mmDia -> Capacitors_SMD:C_0805
- C3: value .1uF -> 10000pF
- C54, C55, C59, C60, C61: value .1uF -> 10uF; footprint Capacitors_SMD:C_0603 -> Capacitors_SMD:C_0805
- R15: value 2.7k -> 10k
- R16, R23, R37, R44, R9: value 1k -> Rt
- R17, R24, R31, R38: value 10k -> Rt
- R20, R25, R35, R40: value Rt -> 10k
- R22, R29, R36, R43, R8: value 2.7k -> Rt
- R30: value 1k -> 10k
- R52: value 10k -> 150R
- U10, U12, U14, U16, U4, U6, U8: value THS4524IDBTR -> AD9219; footprint Housings_SSOP:TSSOP-38_4.4x9.7mm_Pitch0.5mm -> extras:QFN-48-1EP
- U11, U13, U15, U17, U5, U7, U9: value AD9219 -> THS4524IDBTR; footprint SMD_Packages:QFN-48-1EP -> Housings_SSOP:TSSOP-38_4.4x9.7mm_Pitch0.5mm
- U3: value AD9219 -> THS4524IDBTR; footprint extras:QFN-48-1EP -> Housings_SSOP:TSSOP-38_4.4x9.7mm_Pitch0.5mm
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- renumbered C1 to C4, C88 to C53, C74 to C56, C75 to C57, C76 to C58, C80 to C62, C81 to C63, C82 to C64, C83 to C65, C84 to C66, C85 to C67, C86 to C68, C87 to C69, R1 to R3, R2 to R4, R60 to R46, R61 to R47, R62 to R48, R63 to R49, R3 to R5, R64 to R50, R65 to R51, U22 to U1, U1 to U2, U18 to U21, U19 to U22, U20 to U23
Connections:
- C10 pad 1: GNDana -> GND
- C11 pad 1: 3V3ana -> Net-(C11-Pad1)
- C11 pad 2: GNDana -> /Frontend/ADC_CLK-
- C12 pad 1: 3V3ana -> Net-(C12-Pad1)
- C12 pad 2: GNDana -> /Frontend/ADC_CLK+
- C13 pad 1: /Frontend/ADCChannel2/VOCM -> Net-(C13-Pad1)
- C13 pad 2: GNDana -> GND
- C14 pad 1: Net-(C14-Pad1) -> Net-(C13-Pad1)
- C14 pad 2: /Frontend/ADC_CLK- -> Net-(C14-Pad2)
- C15 pad 1: Net-(C15-Pad1) -> Net-(C14-Pad2)
- C15 pad 2: /Frontend/ADC_CLK+ -> Net-(C13-Pad1)
- C16 pad 1: Net-(C16-Pad1) -> GND
- C16 pad 2: GNDana -> Net-(C14-Pad2)
- C17 pad 1: Net-(C16-Pad1) -> Net-(C17-Pad1)
- C17 pad 2: Net-(C17-Pad2) -> /Frontend/ADC_CLK-
- C18 pad 1: Net-(C17-Pad2) -> Net-(C18-Pad1)
- C18 pad 2: Net-(C16-Pad1) -> /Frontend/ADC_CLK+
- C19 pad 1: GNDana -> Net-(C19-Pad1)
- C19 pad 2: Net-(C17-Pad2) -> GND
- C2 pad 2: GNDana -> GND
- C20 pad 1: 3V3ana -> Net-(C19-Pad1)
- C20 pad 2: GNDana -> Net-(C20-Pad2)
- C21 pad 1: 3V3ana -> Net-(C20-Pad2)
- C21 pad 2: GNDana -> Net-(C19-Pad1)
- C22 pad 1: /Frontend/ADCChannel4/VOCM -> GND
- C22 pad 2: GNDana -> Net-(C20-Pad2)
- C25 pad 2: GNDana -> GND
- C28 pad 1: GNDana -> GND
- C29 pad 1: 3V3ana -> Net-(C29-Pad1)
- C29 pad 2: GNDana -> /Frontend/ADC_CLK-
- C3 pad 1: 3V3ana -> /Frontend/ADCChannel1/Vocm
- C3 pad 2: GNDana -> GND
- C30 pad 1: 3V3ana -> Net-(C30-Pad1)
- C30 pad 2: GNDana -> /Frontend/ADC_CLK+
- C31 pad 1: /Frontend/ADCChannel3/VOCM -> Net-(C31-Pad1)
- C31 pad 2: GNDana -> GND
- C32 pad 1: Net-(C32-Pad1) -> Net-(C31-Pad1)
- C32 pad 2: /Frontend/ADC_CLK- -> Net-(C32-Pad2)
- C33 pad 1: Net-(C33-Pad1) -> Net-(C32-Pad2)
- C33 pad 2: /Frontend/ADC_CLK+ -> Net-(C31-Pad1)
- C34 pad 1: Net-(C34-Pad1) -> GND
- C34 pad 2: GNDana -> Net-(C32-Pad2)
- C35 pad 1: Net-(C34-Pad1) -> Net-(C35-Pad1)
- C35 pad 2: Net-(C35-Pad2) -> /Frontend/ADC_CLK-
- C36 pad 1: Net-(C35-Pad2) -> Net-(C36-Pad1)
- C36 pad 2: Net-(C34-Pad1) -> /Frontend/ADC_CLK+
- C37 pad 1: GNDana -> Net-(C37-Pad1)
- C37 pad 2: Net-(C35-Pad2) -> GND
- C38 pad 1: 3V3ana -> Net-(C37-Pad1)
- C38 pad 2: GNDana -> Net-(C38-Pad2)
- C39 pad 1: 3V3ana -> Net-(C38-Pad2)
- C39 pad 2: GNDana -> Net-(C37-Pad1)
- C40 pad 1: /Frontend/ADCChannel8/VOCM -> GND
- C40 pad 2: GNDana -> Net-(C38-Pad2)
- C43 pad 2: GNDana -> GND
- C46 pad 1: GNDana -> GND
- C47 pad 1: 3V3ana -> Net-(C47-Pad1)
- C47 pad 2: GNDana -> /Frontend/ADC_CLK-
- C48 pad 1: 3V3ana -> Net-(C48-Pad1)
- C48 pad 2: GNDana -> /Frontend/ADC_CLK+
- C49 pad 1: /Frontend/ADCChannel7/VOCM -> Net-(C49-Pad1)
- C49 pad 2: GNDana -> GND
- C50 pad 1: Net-(C50-Pad1) -> Net-(C49-Pad1)
- C50 pad 2: /Frontend/ADC_CLK- -> Net-(C50-Pad2)
- C51 pad 1: Net-(C51-Pad1) -> Net-(C50-Pad2)
- C51 pad 2: /Frontend/ADC_CLK+ -> Net-(C49-Pad1)
- C52 pad 1: Net-(C52-Pad1) -> GND
- C52 pad 2: GNDana -> Net-(C50-Pad2)
- C53 pad 1: /Power/5Vraw -> Net-(C53-Pad1)
- C53 pad 2: GNDdig -> GND
- C54 pad 1: Net-(C53-Pad2) -> Net-(C53-Pad1)
- C54 pad 2: Net-(C52-Pad1) -> GND
- C55 pad 1: GNDana -> /Power/5Vdig
- C55 pad 2: Net-(C53-Pad2) -> GND
- C56 pad 1: /Power/5Vraw -> /Power/5Vdig
- C57 pad 1: /Power/5Vraw -> /Power/5Vdig
- C58 pad 1: /Power/5Vraw -> /Power/5Vdig
- C59 pad 1: Net-(C59-Pad1) -> /Power/5Vdig
- C59 pad 2: /Frontend/ADC_CLK- -> GNDdig
- C60 pad 1: Net-(C60-Pad1) -> /Power/5Vdig
- C60 pad 2: /Frontend/ADC_CLK+ -> GNDdig
- C61 pad 1: Net-(C61-Pad1) -> /Power/5Vdig
- C61 pad 2: GNDana -> GNDdig
- C7 pad 2: GNDana -> GND
- CON1 pad 1: /Power/5Vraw -> Net-(CON1-Pad1)
- CON1 pad 2: GNDdig -> Net-(CON1-Pad2)
- CON1 pad 3: GNDdig -> Net-(CON1-Pad2)
- P3 pad 11: 5Vdig -> (no net)
- R10 pad 1: GNDana -> GND
- R11 pad 1: /Frontend/ADCChannel2/EXT_CHA+ -> /Frontend/ADCChannel4/EXT_CHA+
- R11 pad 2: /Frontend/ADCChannel2/EXT_CHA- -> /Frontend/ADCChannel4/EXT_CHA-
- R12 pad 1: /Frontend/ADCChannel2/EXT_CHB+ -> /Frontend/ADCChannel4/EXT_CHB+
- R12 pad 2: /Frontend/ADCChannel2/EXT_CHB- -> /Frontend/ADCChannel4/EXT_CHB-
- R13 pad 1: /Frontend/ADCChannel2/EXT_CHC+ -> /Frontend/ADCChannel4/EXT_CHC+
- R13 pad 2: /Frontend/ADCChannel2/EXT_CHC- -> /Frontend/ADCChannel4/EXT_CHC-
- R14 pad 1: /Frontend/ADCChannel2/EXT_CHD+ -> /Frontend/ADCChannel4/EXT_CHD+
- R14 pad 2: /Frontend/ADCChannel2/EXT_CHD- -> /Frontend/ADCChannel4/EXT_CHD-
- R15 pad 1: 3V3ana -> GND
- R15 pad 2: /Frontend/ADCChannel2/VOCM -> Net-(R15-Pad2)
- R16 pad 1: /Frontend/ADCChannel2/VOCM -> /Frontend/ADCChannel3/EXT_CHA+
- R16 pad 2: GNDana -> /Frontend/ADCChannel3/EXT_CHA-
- R17 pad 1: GNDana -> /Frontend/ADCChannel3/EXT_CHB+
- R17 pad 2: Net-(R17-Pad2) -> /Frontend/ADCChannel3/EXT_CHB-
- R18 pad 1: /Frontend/ADCChannel4/EXT_CHA+ -> /Frontend/ADCChannel3/EXT_CHC+
- R18 pad 2: /Frontend/ADCChannel4/EXT_CHA- -> /Frontend/ADCChannel3/EXT_CHC-
- R19 pad 1: /Frontend/ADCChannel4/EXT_CHB+ -> /Frontend/ADCChannel3/EXT_CHD+
- R19 pad 2: /Frontend/ADCChannel4/EXT_CHB- -> /Frontend/ADCChannel3/EXT_CHD-
- R20 pad 1: /Frontend/ADCChannel4/EXT_CHC+ -> GND
- R20 pad 2: /Frontend/ADCChannel4/EXT_CHC- -> Net-(R20-Pad2)
- R21 pad 1: /Frontend/ADCChannel4/EXT_CHD+ -> /Frontend/ADCChannel8/EXT_CHA+
- R21 pad 2: /Frontend/ADCChannel4/EXT_CHD- -> /Frontend/ADCChannel8/EXT_CHA-
- R22 pad 1: 3V3ana -> /Frontend/ADCChannel8/EXT_CHB+
- R22 pad 2: /Frontend/ADCChannel4/VOCM -> /Frontend/ADCChannel8/EXT_CHB-
- R23 pad 1: /Frontend/ADCChannel4/VOCM -> /Frontend/ADCChannel8/EXT_CHC+
- R23 pad 2: GNDana -> /Frontend/ADCChannel8/EXT_CHC-
- R24 pad 1: GNDana -> /Frontend/ADCChannel8/EXT_CHD+
- R24 pad 2: Net-(R24-Pad2) -> /Frontend/ADCChannel8/EXT_CHD-
- R25 pad 1: /Frontend/ADCChannel3/EXT_CHA+ -> GND
- R25 pad 2: /Frontend/ADCChannel3/EXT_CHA- -> Net-(R25-Pad2)
- R26 pad 1: /Frontend/ADCChannel3/EXT_CHB+ -> /Frontend/ADCChannel7/EXT_CHA+
- R26 pad 2: /Frontend/ADCChannel3/EXT_CHB- -> /Frontend/ADCChannel7/EXT_CHA-
- R27 pad 1: /Frontend/ADCChannel3/EXT_CHC+ -> /Frontend/ADCChannel7/EXT_CHB+
- R27 pad 2: /Frontend/ADCChannel3/EXT_CHC- -> /Frontend/ADCChannel7/EXT_CHB-
- R28 pad 1: /Frontend/ADCChannel3/EXT_CHD+ -> /Frontend/ADCChannel7/EXT_CHC+
- R28 pad 2: /Frontend/ADCChannel3/EXT_CHD- -> /Frontend/ADCChannel7/EXT_CHC-
- R29 pad 1: 3V3ana -> /Frontend/ADCChannel7/EXT_CHD+
- R29 pad 2: /Frontend/ADCChannel3/VOCM -> /Frontend/ADCChannel7/EXT_CHD-
- R30 pad 1: /Frontend/ADCChannel3/VOCM -> GND
- R30 pad 2: GNDana -> Net-(R30-Pad2)
- R31 pad 1: GNDana -> /Frontend/ADCChannel5/EXT_CHA+
- R31 pad 2: Net-(R31-Pad2) -> /Frontend/ADCChannel5/EXT_CHA-
- R32 pad 1: /Frontend/ADCChannel8/EXT_CHA+ -> /Frontend/ADCChannel5/EXT_CHB+
- R32 pad 2: /Frontend/ADCChannel8/EXT_CHA- -> /Frontend/ADCChannel5/EXT_CHB-
- R33 pad 1: /Frontend/ADCChannel8/EXT_CHB+ -> /Frontend/ADCChannel5/EXT_CHC+
- R33 pad 2: /Frontend/ADCChannel8/EXT_CHB- -> /Frontend/ADCChannel5/EXT_CHC-
- R34 pad 1: /Frontend/ADCChannel8/EXT_CHC+ -> /Frontend/ADCChannel5/EXT_CHD+
- R34 pad 2: /Frontend/ADCChannel8/EXT_CHC- -> /Frontend/ADCChannel5/EXT_CHD-
- R35 pad 1: /Frontend/ADCChannel8/EXT_CHD+ -> GND
- R35 pad 2: /Frontend/ADCChannel8/EXT_CHD- -> Net-(R35-Pad2)
- R36 pad 1: 3V3ana -> /Frontend/ADCChannel6/EXT_CHA+
- R36 pad 2: /Frontend/ADCChannel8/VOCM -> /Frontend/ADCChannel6/EXT_CHA-
- R37 pad 1: /Frontend/ADCChannel8/VOCM -> /Frontend/ADCChannel6/EXT_CHB+
- R37 pad 2: GNDana -> /Frontend/ADCChannel6/EXT_CHB-
- R38 pad 1: GNDana -> /Frontend/ADCChannel6/EXT_CHC+
- R38 pad 2: Net-(R38-Pad2) -> /Frontend/ADCChannel6/EXT_CHC-
- R39 pad 1: /Frontend/ADCChannel7/EXT_CHA+ -> /Frontend/ADCChannel6/EXT_CHD+
- R39 pad 2: /Frontend/ADCChannel7/EXT_CHA- -> /Frontend/ADCChannel6/EXT_CHD-
- R40 pad 1: /Frontend/ADCChannel7/EXT_CHB+ -> GND
- R40 pad 2: /Frontend/ADCChannel7/EXT_CHB- -> Net-(R40-Pad2)
- R41 pad 1: /Frontend/ADCChannel7/EXT_CHC+ -> /Frontend/ADCChannel2/EXT_CHA+
- R41 pad 2: /Frontend/ADCChannel7/EXT_CHC- -> /Frontend/ADCChannel2/EXT_CHA-
- R42 pad 1: /Frontend/ADCChannel7/EXT_CHD+ -> /Frontend/ADCChannel2/EXT_CHB+
- R42 pad 2: /Frontend/ADCChannel7/EXT_CHD- -> /Frontend/ADCChannel2/EXT_CHB-
- R43 pad 1: 3V3ana -> /Frontend/ADCChannel2/EXT_CHC+
- R43 pad 2: /Frontend/ADCChannel7/VOCM -> /Frontend/ADCChannel2/EXT_CHC-
- R44 pad 1: /Frontend/ADCChannel7/VOCM -> /Frontend/ADCChannel2/EXT_CHD+
- R44 pad 2: GNDana -> /Frontend/ADCChannel2/EXT_CHD-
- R45 pad 1: GNDana -> GND
- R52 pad 1: GNDana -> /Power/5Vdig
- R52 pad 2: Net-(R52-Pad2) -> Net-(D1-Pad2)
- R6 pad 1: /Frontend/ADCChannel1/EXT_CHC+ -> /Frontend/ADCChannel1/EXT_CHA+
- R6 pad 2: /Frontend/ADCChannel1/EXT_CHC- -> /Frontend/ADCChannel1/EXT_CHA-
- R7 pad 1: /Frontend/ADCChannel1/EXT_CHD+ -> /Frontend/ADCChannel1/EXT_CHB+
- R7 pad 2: /Frontend/ADCChannel1/EXT_CHD- -> /Frontend/ADCChannel1/EXT_CHB-
- R8 pad 1: 3V3ana -> /Frontend/ADCChannel1/EXT_CHC+
- R8 pad 2: /Frontend/ADCChannel1/VOCM -> /Frontend/ADCChannel1/EXT_CHC-
- R9 pad 1: /Frontend/ADCChannel1/VOCM -> /Frontend/ADCChannel1/EXT_CHD+
- R9 pad 2: GNDana -> /Frontend/ADCChannel1/EXT_CHD-
- RP10 pad 1: /Frontend/ADCChannel3/EXT_CHA+ -> /Frontend/ADCChannel8/EXT_CHA+
- RP10 pad 2: /Frontend/ADCChannel3/EXT_CHA- -> /Frontend/ADCChannel8/EXT_CHA-
- RP10 pad 3: /Frontend/ADCChannel3/EXT_CHB+ -> /Frontend/ADCChannel8/EXT_CHB+
- RP10 pad 4: /Frontend/ADCChannel3/EXT_CHB- -> /Frontend/ADCChannel8/EXT_CHB-
- RP10 pad 5: /Frontend/ADCChannel3/EXT_CHC+ -> /Frontend/ADCChannel8/EXT_CHC+
- RP10 pad 6: /Frontend/ADCChannel3/EXT_CHC- -> /Frontend/ADCChannel8/EXT_CHC-
- RP10 pad 7: /Frontend/ADCChannel3/EXT_CHD+ -> /Frontend/ADCChannel8/EXT_CHD+
- RP10 pad 8: /Frontend/ADCChannel3/EXT_CHD- -> /Frontend/ADCChannel8/EXT_CHD-
- RP11 pad 1: Net-(RP10-Pad10) -> Net-(RP10-Pad12)
- RP11 pad 2: Net-(RP10-Pad9) -> Net-(RP10-Pad11)
- RP11 pad 3: Net-(RP10-Pad12) -> Net-(RP10-Pad10)
- RP11 pad 4: Net-(RP10-Pad11) -> Net-(RP10-Pad9)
- RP11 pad 5: /Frontend/ADCChannel3/CHC- -> /Frontend/ADCChannel8/CHC-
- RP11 pad 6: /Frontend/ADCChannel3/CHC+ -> /Frontend/ADCChannel8/CHC+
- RP11 pad 7: /Frontend/ADCChannel3/CHD- -> /Frontend/ADCChannel8/CHD-
- RP11 pad 8: /Frontend/ADCChannel3/CHD+ -> /Frontend/ADCChannel8/CHD+
- RP12 pad 1: Net-(RP10-Pad14) -> Net-(RP10-Pad16)
- RP12 pad 2: Net-(RP10-Pad13) -> Net-(RP10-Pad15)
- RP12 pad 3: Net-(RP10-Pad16) -> Net-(RP10-Pad14)
- RP12 pad 4: Net-(RP10-Pad15) -> Net-(RP10-Pad13)
- RP12 pad 5: /Frontend/ADCChannel3/CHA- -> /Frontend/ADCChannel8/CHA-
- RP12 pad 6: /Frontend/ADCChannel3/CHA+ -> /Frontend/ADCChannel8/CHA+
- RP12 pad 7: /Frontend/ADCChannel3/CHB- -> /Frontend/ADCChannel8/CHB-
- RP12 pad 8: /Frontend/ADCChannel3/CHB+ -> /Frontend/ADCChannel8/CHB+
- RP13 pad 1: /Frontend/ADCChannel8/EXT_CHA+ -> /Frontend/ADCChannel7/EXT_CHA+
- RP13 pad 2: /Frontend/ADCChannel8/EXT_CHA- -> /Frontend/ADCChannel7/EXT_CHA-
- RP13 pad 3: /Frontend/ADCChannel8/EXT_CHB+ -> /Frontend/ADCChannel7/EXT_CHB+
- RP13 pad 4: /Frontend/ADCChannel8/EXT_CHB- -> /Frontend/ADCChannel7/EXT_CHB-
- RP13 pad 5: /Frontend/ADCChannel8/EXT_CHC+ -> /Frontend/ADCChannel7/EXT_CHC+
- RP13 pad 6: /Frontend/ADCChannel8/EXT_CHC- -> /Frontend/ADCChannel7/EXT_CHC-
- RP13 pad 7: /Frontend/ADCChannel8/EXT_CHD+ -> /Frontend/ADCChannel7/EXT_CHD+
- RP13 pad 8: /Frontend/ADCChannel8/EXT_CHD- -> /Frontend/ADCChannel7/EXT_CHD-
- RP14 pad 1: Net-(RP13-Pad10) -> Net-(RP13-Pad12)
- RP14 pad 2: Net-(RP13-Pad9) -> Net-(RP13-Pad11)
- RP14 pad 3: Net-(RP13-Pad12) -> Net-(RP13-Pad10)
- RP14 pad 4: Net-(RP13-Pad11) -> Net-(RP13-Pad9)
- RP14 pad 5: /Frontend/ADCChannel8/CHC- -> /Frontend/ADCChannel7/CHC-
- RP14 pad 6: /Frontend/ADCChannel8/CHC+ -> /Frontend/ADCChannel7/CHC+
- RP14 pad 7: /Frontend/ADCChannel8/CHD- -> /Frontend/ADCChannel7/CHD-
- RP14 pad 8: /Frontend/ADCChannel8/CHD+ -> /Frontend/ADCChannel7/CHD+
- RP15 pad 1: Net-(RP13-Pad14) -> Net-(RP13-Pad16)
- RP15 pad 2: Net-(RP13-Pad13) -> Net-(RP13-Pad15)
- RP15 pad 3: Net-(RP13-Pad16) -> Net-(RP13-Pad14)
- RP15 pad 4: Net-(RP13-Pad15) -> Net-(RP13-Pad13)
- RP15 pad 5: /Frontend/ADCChannel8/CHA- -> /Frontend/ADCChannel7/CHA-
- RP15 pad 6: /Frontend/ADCChannel8/CHA+ -> /Frontend/ADCChannel7/CHA+
- RP15 pad 7: /Frontend/ADCChannel8/CHB- -> /Frontend/ADCChannel7/CHB-
- RP15 pad 8: /Frontend/ADCChannel8/CHB+ -> /Frontend/ADCChannel7/CHB+
- RP16 pad 1: /Frontend/ADCChannel7/EXT_CHA+ -> /Frontend/ADCChannel5/EXT_CHA+
- RP16 pad 2: /Frontend/ADCChannel7/EXT_CHA- -> /Frontend/ADCChannel5/EXT_CHA-
- RP16 pad 3: /Frontend/ADCChannel7/EXT_CHB+ -> /Frontend/ADCChannel5/EXT_CHB+
- RP16 pad 4: /Frontend/ADCChannel7/EXT_CHB- -> /Frontend/ADCChannel5/EXT_CHB-
- RP16 pad 5: /Frontend/ADCChannel7/EXT_CHC+ -> /Frontend/ADCChannel5/EXT_CHC+
- RP16 pad 6: /Frontend/ADCChannel7/EXT_CHC- -> /Frontend/ADCChannel5/EXT_CHC-
- RP16 pad 7: /Frontend/ADCChannel7/EXT_CHD+ -> /Frontend/ADCChannel5/EXT_CHD+
- RP16 pad 8: /Frontend/ADCChannel7/EXT_CHD- -> /Frontend/ADCChannel5/EXT_CHD-
- RP17 pad 1: Net-(RP16-Pad10) -> Net-(RP16-Pad12)
- RP17 pad 2: Net-(RP16-Pad9) -> Net-(RP16-Pad11)
- RP17 pad 3: Net-(RP16-Pad12) -> Net-(RP16-Pad10)
- RP17 pad 4: Net-(RP16-Pad11) -> Net-(RP16-Pad9)
- RP17 pad 5: /Frontend/ADCChannel7/CHC- -> /Frontend/ADCChannel5/CHC-
- RP17 pad 6: /Frontend/ADCChannel7/CHC+ -> /Frontend/ADCChannel5/CHC+
- RP17 pad 7: /Frontend/ADCChannel7/CHD- -> /Frontend/ADCChannel5/CHD-
- RP17 pad 8: /Frontend/ADCChannel7/CHD+ -> /Frontend/ADCChannel5/CHD+
- RP18 pad 1: Net-(RP16-Pad14) -> Net-(RP16-Pad16)
- RP18 pad 2: Net-(RP16-Pad13) -> Net-(RP16-Pad15)
- RP18 pad 3: Net-(RP16-Pad16) -> Net-(RP16-Pad14)
- RP18 pad 4: Net-(RP16-Pad15) -> Net-(RP16-Pad13)
- RP18 pad 5: /Frontend/ADCChannel7/CHA- -> /Frontend/ADCChannel5/CHA-
- RP18 pad 6: /Frontend/ADCChannel7/CHA+ -> /Frontend/ADCChannel5/CHA+
- RP18 pad 7: /Frontend/ADCChannel7/CHB- -> /Frontend/ADCChannel5/CHB-
- RP18 pad 8: /Frontend/ADCChannel7/CHB+ -> /Frontend/ADCChannel5/CHB+
- RP19 pad 1: /Frontend/ADCChannel5/EXT_CHA+ -> /Frontend/ADCChannel6/EXT_CHA+
- RP19 pad 2: /Frontend/ADCChannel5/EXT_CHA- -> /Frontend/ADCChannel6/EXT_CHA-
- RP19 pad 3: /Frontend/ADCChannel5/EXT_CHB+ -> /Frontend/ADCChannel6/EXT_CHB+
- RP19 pad 4: /Frontend/ADCChannel5/EXT_CHB- -> /Frontend/ADCChannel6/EXT_CHB-
- RP19 pad 5: /Frontend/ADCChannel5/EXT_CHC+ -> /Frontend/ADCChannel6/EXT_CHC+
- RP19 pad 6: /Frontend/ADCChannel5/EXT_CHC- -> /Frontend/ADCChannel6/EXT_CHC-
- RP19 pad 7: /Frontend/ADCChannel5/EXT_CHD+ -> /Frontend/ADCChannel6/EXT_CHD+
- RP19 pad 8: /Frontend/ADCChannel5/EXT_CHD- -> /Frontend/ADCChannel6/EXT_CHD-
- RP20 pad 1: Net-(RP19-Pad10) -> Net-(RP19-Pad12)
- RP20 pad 2: Net-(RP19-Pad9) -> Net-(RP19-Pad11)
- RP20 pad 3: Net-(RP19-Pad12) -> Net-(RP19-Pad10)
- RP20 pad 4: Net-(RP19-Pad11) -> Net-(RP19-Pad9)
- RP20 pad 5: /Frontend/ADCChannel5/CHC- -> /Frontend/ADCChannel6/CHC-
- RP20 pad 6: /Frontend/ADCChannel5/CHC+ -> /Frontend/ADCChannel6/CHC+
- RP20 pad 7: /Frontend/ADCChannel5/CHD- -> /Frontend/ADCChannel6/CHD-
- RP20 pad 8: /Frontend/ADCChannel5/CHD+ -> /Frontend/ADCChannel6/CHD+
- RP21 pad 1: Net-(RP19-Pad14) -> Net-(RP19-Pad16)
- RP21 pad 2: Net-(RP19-Pad13) -> Net-(RP19-Pad15)
- RP21 pad 3: Net-(RP19-Pad16) -> Net-(RP19-Pad14)
- RP21 pad 4: Net-(RP19-Pad15) -> Net-(RP19-Pad13)
- RP21 pad 5: /Frontend/ADCChannel5/CHA- -> /Frontend/ADCChannel6/CHA-
- RP21 pad 6: /Frontend/ADCChannel5/CHA+ -> /Frontend/ADCChannel6/CHA+
- RP21 pad 7: /Frontend/ADCChannel5/CHB- -> /Frontend/ADCChannel6/CHB-
- RP21 pad 8: /Frontend/ADCChannel5/CHB+ -> /Frontend/ADCChannel6/CHB+
- RP22 pad 1: /Frontend/ADCChannel6/EXT_CHA+ -> /Frontend/ADCChannel2/EXT_CHA+
- RP22 pad 2: /Frontend/ADCChannel6/EXT_CHA- -> /Frontend/ADCChannel2/EXT_CHA-
- RP22 pad 3: /Frontend/ADCChannel6/EXT_CHB+ -> /Frontend/ADCChannel2/EXT_CHB+
- RP22 pad 4: /Frontend/ADCChannel6/EXT_CHB- -> /Frontend/ADCChannel2/EXT_CHB-
- RP22 pad 5: /Frontend/ADCChannel6/EXT_CHC+ -> /Frontend/ADCChannel2/EXT_CHC+
- RP22 pad 6: /Frontend/ADCChannel6/EXT_CHC- -> /Frontend/ADCChannel2/EXT_CHC-
- RP22 pad 7: /Frontend/ADCChannel6/EXT_CHD+ -> /Frontend/ADCChannel2/EXT_CHD+
- RP22 pad 8: /Frontend/ADCChannel6/EXT_CHD- -> /Frontend/ADCChannel2/EXT_CHD-
- RP23 pad 1: Net-(RP22-Pad10) -> Net-(RP22-Pad12)
- RP23 pad 2: Net-(RP22-Pad9) -> Net-(RP22-Pad11)
- RP23 pad 3: Net-(RP22-Pad12) -> Net-(RP22-Pad10)
- RP23 pad 4: Net-(RP22-Pad11) -> Net-(RP22-Pad9)
- RP23 pad 5: /Frontend/ADCChannel6/CHC- -> /Frontend/ADCChannel2/CHC-
- RP23 pad 6: /Frontend/ADCChannel6/CHC+ -> /Frontend/ADCChannel2/CHC+
- RP23 pad 7: /Frontend/ADCChannel6/CHD- -> /Frontend/ADCChannel2/CHD-
- RP23 pad 8: /Frontend/ADCChannel6/CHD+ -> /Frontend/ADCChannel2/CHD+
- RP24 pad 1: Net-(RP22-Pad14) -> Net-(RP22-Pad16)
- RP24 pad 2: Net-(RP22-Pad13) -> Net-(RP22-Pad15)
- RP24 pad 3: Net-(RP22-Pad16) -> Net-(RP22-Pad14)
- RP24 pad 4: Net-(RP22-Pad15) -> Net-(RP22-Pad13)
- RP24 pad 5: /Frontend/ADCChannel6/CHA- -> /Frontend/ADCChannel2/CHA-
- RP24 pad 6: /Frontend/ADCChannel6/CHA+ -> /Frontend/ADCChannel2/CHA+
- RP24 pad 7: /Frontend/ADCChannel6/CHB- -> /Frontend/ADCChannel2/CHB-
- RP24 pad 8: /Frontend/ADCChannel6/CHB+ -> /Frontend/ADCChannel2/CHB+
- RP4 pad 1: /Frontend/ADCChannel2/EXT_CHA+ -> /Frontend/ADCChannel4/EXT_CHA+
- RP4 pad 2: /Frontend/ADCChannel2/EXT_CHA- -> /Frontend/ADCChannel4/EXT_CHA-
- RP4 pad 3: /Frontend/ADCChannel2/EXT_CHB+ -> /Frontend/ADCChannel4/EXT_CHB+
- RP4 pad 4: /Frontend/ADCChannel2/EXT_CHB- -> /Frontend/ADCChannel4/EXT_CHB-
- RP4 pad 5: /Frontend/ADCChannel2/EXT_CHC+ -> /Frontend/ADCChannel4/EXT_CHC+
- RP4 pad 6: /Frontend/ADCChannel2/EXT_CHC- -> /Frontend/ADCChannel4/EXT_CHC-
- RP4 pad 7: /Frontend/ADCChannel2/EXT_CHD+ -> /Frontend/ADCChannel4/EXT_CHD+
- RP4 pad 8: /Frontend/ADCChannel2/EXT_CHD- -> /Frontend/ADCChannel4/EXT_CHD-
- RP5 pad 1: Net-(RP4-Pad10) -> Net-(RP4-Pad12)
- RP5 pad 2: Net-(RP4-Pad9) -> Net-(RP4-Pad11)
- RP5 pad 3: Net-(RP4-Pad12) -> Net-(RP4-Pad10)
- RP5 pad 4: Net-(RP4-Pad11) -> Net-(RP4-Pad9)
- RP5 pad 5: /Frontend/ADCChannel2/CHC- -> /Frontend/ADCChannel4/CHC-
- RP5 pad 6: /Frontend/ADCChannel2/CHC+ -> /Frontend/ADCChannel4/CHC+
- RP5 pad 7: /Frontend/ADCChannel2/CHD- -> /Frontend/ADCChannel4/CHD-
- RP5 pad 8: /Frontend/ADCChannel2/CHD+ -> /Frontend/ADCChannel4/CHD+
- RP6 pad 1: Net-(RP4-Pad14) -> Net-(RP4-Pad16)
- RP6 pad 2: Net-(RP4-Pad13) -> Net-(RP4-Pad15)
- RP6 pad 3: Net-(RP4-Pad16) -> Net-(RP4-Pad14)
- RP6 pad 4: Net-(RP4-Pad15) -> Net-(RP4-Pad13)
- RP6 pad 5: /Frontend/ADCChannel2/CHA- -> /Frontend/ADCChannel4/CHA-
- RP6 pad 6: /Frontend/ADCChannel2/CHA+ -> /Frontend/ADCChannel4/CHA+
- RP6 pad 7: /Frontend/ADCChannel2/CHB- -> /Frontend/ADCChannel4/CHB-
- RP6 pad 8: /Frontend/ADCChannel2/CHB+ -> /Frontend/ADCChannel4/CHB+
- RP7 pad 1: /Frontend/ADCChannel4/EXT_CHA+ -> /Frontend/ADCChannel3/EXT_CHA+
- RP7 pad 2: /Frontend/ADCChannel4/EXT_CHA- -> /Frontend/ADCChannel3/EXT_CHA-
- RP7 pad 3: /Frontend/ADCChannel4/EXT_CHB+ -> /Frontend/ADCChannel3/EXT_CHB+
- RP7 pad 4: /Frontend/ADCChannel4/EXT_CHB- -> /Frontend/ADCChannel3/EXT_CHB-
- RP7 pad 5: /Frontend/ADCChannel4/EXT_CHC+ -> /Frontend/ADCChannel3/EXT_CHC+
- RP7 pad 6: /Frontend/ADCChannel4/EXT_CHC- -> /Frontend/ADCChannel3/EXT_CHC-
- RP7 pad 7: /Frontend/ADCChannel4/EXT_CHD+ -> /Frontend/ADCChannel3/EXT_CHD+
- RP7 pad 8: /Frontend/ADCChannel4/EXT_CHD- -> /Frontend/ADCChannel3/EXT_CHD-
- RP8 pad 1: Net-(RP7-Pad10) -> Net-(RP7-Pad12)
- RP8 pad 2: Net-(RP7-Pad9) -> Net-(RP7-Pad11)
- RP8 pad 3: Net-(RP7-Pad12) -> Net-(RP7-Pad10)
- RP8 pad 4: Net-(RP7-Pad11) -> Net-(RP7-Pad9)
- RP8 pad 5: /Frontend/ADCChannel4/CHC- -> /Frontend/ADCChannel3/CHC-
- RP8 pad 6: /Frontend/ADCChannel4/CHC+ -> /Frontend/ADCChannel3/CHC+
- RP8 pad 7: /Frontend/ADCChannel4/CHD- -> /Frontend/ADCChannel3/CHD-
- RP8 pad 8: /Frontend/ADCChannel4/CHD+ -> /Frontend/ADCChannel3/CHD+
- RP9 pad 1: Net-(RP7-Pad14) -> Net-(RP7-Pad16)
- RP9 pad 2: Net-(RP7-Pad13) -> Net-(RP7-Pad15)
- RP9 pad 3: Net-(RP7-Pad16) -> Net-(RP7-Pad14)
- RP9 pad 4: Net-(RP7-Pad15) -> Net-(RP7-Pad13)
- RP9 pad 5: /Frontend/ADCChannel4/CHA- -> /Frontend/ADCChannel3/CHA-
- RP9 pad 6: /Frontend/ADCChannel4/CHA+ -> /Frontend/ADCChannel3/CHA+
- RP9 pad 7: /Frontend/ADCChannel4/CHB- -> /Frontend/ADCChannel3/CHB-
- RP9 pad 8: /Frontend/ADCChannel4/CHB+ -> /Frontend/ADCChannel3/CHB+
- U10 pad 1: (no net) -> 1V8ana
- U10 pad 10: GNDana -> 1V8ana
- U10 pad 11: (no net) -> GND
- U10 pad 12: Net-(RP13-Pad12) -> 1V8dig
- U10 pad 13: Net-(RP13-Pad11) -> (no net)
- U10 pad 14: /Frontend/ADCChannel8/VOCM -> (no net)
- U10 pad 15: GNDana -> (no net)
- U10 pad 17: Net-(RP13-Pad10) -> (no net)
- U10 pad 18: Net-(RP13-Pad9) -> (no net)
- U10 pad 19: /Frontend/ADCChannel8/VOCM -> (no net)
- U10 pad 2: Net-(RP13-Pad16) -> 1V8ana
- U10 pad 20: 3V3ana -> (no net)
- U10 pad 21: /Frontend/ADCChannel8/CHD+ -> (no net)
- U10 pad 22: /Frontend/ADCChannel8/CHD- -> (no net)
- U10 pad 23: GNDana -> (no net)
- U10 pad 24: GNDana -> (no net)
- U10 pad 25: 3V3ana -> 1V8dig
- U10 pad 26: /Frontend/ADCChannel8/CHC+ -> GND
- U10 pad 27: /Frontend/ADCChannel8/CHC- -> 1V8ana
- U10 pad 28: GNDana -> /Frontend/ADC_SCLK
- U10 pad 29: GNDana -> /Frontend/ADC_SDIO
- U10 pad 3: Net-(RP13-Pad15) -> /Frontend/ADCChannel8/CHD-
- U10 pad 30: 3V3ana -> (no net)
- U10 pad 31: /Frontend/ADCChannel8/CHB+ -> GND
- U10 pad 32: /Frontend/ADCChannel8/CHB- -> 1V8ana
- U10 pad 33: GNDana -> /Frontend/ADCChannel8/CHA+
- U10 pad 34: GNDana -> /Frontend/ADCChannel8/CHA-
- U10 pad 35: 3V3ana -> 1V8ana
- U10 pad 36: /Frontend/ADCChannel8/CHA+ -> 1V8ana
- U10 pad 37: /Frontend/ADCChannel8/CHA- -> /Frontend/ADCChannel8/CHB-
- U10 pad 38: GNDana -> /Frontend/ADCChannel8/CHB+
- U10 pad 4: /Frontend/ADCChannel8/VOCM -> /Frontend/ADCChannel8/CHD+
- U10 pad 5: GNDana -> 1V8ana
- U10 pad 6: (no net) -> 1V8ana
- U10 pad 7: Net-(RP13-Pad14) -> Net-(C23-Pad1)
- U10 pad 8: Net-(RP13-Pad13) -> Net-(C24-Pad1)
- U10 pad 9: /Frontend/ADCChannel8/VOCM -> 1V8ana
- U11 pad 1: 1V8ana -> (no net)
- U11 pad 10: 1V8ana -> GND
- U11 pad 11: GNDdig -> (no net)
- U11 pad 12: 1V8dig -> Net-(RP13-Pad12)
- U11 pad 13: (no net) -> Net-(RP13-Pad11)
- U11 pad 14: (no net) -> /Frontend/ADCChannel1/Vocm
- U11 pad 15: (no net) -> GND
- U11 pad 17: (no net) -> Net-(RP13-Pad10)
- U11 pad 18: (no net) -> Net-(RP13-Pad9)
- U11 pad 19: (no net) -> /Frontend/ADCChannel1/Vocm
- U11 pad 2: 1V8ana -> Net-(RP13-Pad16)
- U11 pad 20: (no net) -> 3V3ana
- U11 pad 21: (no net) -> /Frontend/ADCChannel7/CHD+
- U11 pad 22: (no net) -> /Frontend/ADCChannel7/CHD-
- U11 pad 23: (no net) -> GND
- U11 pad 24: (no net) -> GND
- U11 pad 25: 1V8dig -> 3V3ana
- U11 pad 26: GNDdig -> /Frontend/ADCChannel7/CHC+
- U11 pad 27: 1V8ana -> /Frontend/ADCChannel7/CHC-
- U11 pad 28: /Frontend/ADC_SCLK -> GND
- U11 pad 29: /Frontend/ADC_SDIO -> GND
- U11 pad 3: /Frontend/ADCChannel8/CHD- -> Net-(RP13-Pad15)
- U11 pad 30: (no net) -> 3V3ana
- U11 pad 31: GNDdig -> /Frontend/ADCChannel7/CHB+
- U11 pad 32: 1V8ana -> /Frontend/ADCChannel7/CHB-
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Routing:
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
Commit message: ADC channels wired, fan controller added
Parts:
- moved R21 329.4 mm to (256.6, 33.7), turned to 180 degrees
- moved C26 326.0 mm to (258.9, 55.4)
- moved R22 325.8 mm to (253.6, 33.7), turned to 180 degrees
- moved R23 322.3 mm to (250.6, 33.7), turned to 180 degrees
- moved R24 321.3 mm to (247.6, 33.7), turned to 180 degrees
- moved C27 318.8 mm to (258.9, 53.4)
- moved C28 315.5 mm to (259.9, 58.2), turned to 90 degrees
- moved C25 313.5 mm to (257.9, 58.2), turned to 270 degrees
- moved C24 310.7 mm to (245.6, 58.3), turned to 270 degrees
- moved C31 305.4 mm to (237.4, 57.9), turned to 270 degrees
- moved C23 303.6 mm to (243.8, 58.3), turned to 270 degrees
- moved C33 301.1 mm to (238.3, 53.1), turned to 180 degrees
- moved C30 298.8 mm to (225.0, 58.0), turned to 270 degrees
- moved C29 292.1 mm to (223.2, 58.0), turned to 270 degrees
- moved C34 287.8 mm to (239.4, 57.9), turned to 90 degrees
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Connections:
- R3 pad 1: /Frontend/ADC_CLK+ -> /Frontend/ADC_CLK-
- R3 pad 2: /Frontend/ADC_CLK- -> /Frontend/ADC_CLK+
- U1 pad 13: /Frontend/ADCChannel8/EXT_CHD- -> /Frontend/ADCChannel2/EXT_CHD-
- U1 pad 14: /Frontend/ADCChannel8/EXT_CHD+ -> /Frontend/ADCChannel2/EXT_CHD+
- U1 pad 15: /Frontend/ADCChannel8/EXT_CHC- -> /Frontend/ADCChannel2/EXT_CHC-
- U1 pad 16: /Frontend/ADCChannel8/EXT_CHC+ -> /Frontend/ADCChannel2/EXT_CHB-
- U1 pad 17: /Frontend/ADCChannel8/EXT_CHB- -> /Frontend/ADCChannel2/EXT_CHB+
- U1 pad 18: /Frontend/ADCChannel8/EXT_CHB+ -> /Frontend/ADCChannel2/EXT_CHC+
- U1 pad 19: /Frontend/ADCChannel8/EXT_CHA- -> /Frontend/ADCChannel2/EXT_CHA-
- U1 pad 20: /Frontend/ADCChannel8/EXT_CHA+ -> /Frontend/ADCChannel2/EXT_CHA+
- U1 pad 25: /Frontend/ADCChannel2/EXT_CHD- -> /Frontend/ADCChannel3/EXT_CHD-
- U1 pad 26: /Frontend/ADCChannel2/EXT_CHD+ -> /Frontend/ADCChannel3/EXT_CHD+
- U1 pad 27: /Frontend/ADCChannel2/EXT_CHC- -> /Frontend/ADCChannel3/EXT_CHC-
- U1 pad 28: /Frontend/ADCChannel2/EXT_CHC+ -> /Frontend/ADCChannel3/EXT_CHB-
- U1 pad 29: /Frontend/ADCChannel2/EXT_CHB- -> /Frontend/ADCChannel3/EXT_CHB+
- U1 pad 30: /Frontend/ADCChannel2/EXT_CHB+ -> /Frontend/ADCChannel3/EXT_CHC+
- U1 pad 31: /Frontend/ADCChannel2/EXT_CHA- -> /Frontend/ADCChannel3/EXT_CHA-
- U1 pad 32: /Frontend/ADCChannel2/EXT_CHA+ -> /Frontend/ADCChannel3/EXT_CHA+
- U1 pad 37: /Frontend/ADCChannel7/EXT_CHD- -> /Frontend/ADCChannel4/EXT_CHD-
- U1 pad 38: /Frontend/ADCChannel7/EXT_CHD+ -> /Frontend/ADCChannel4/EXT_CHD+
- U1 pad 39: /Frontend/ADCChannel7/EXT_CHC- -> /Frontend/ADCChannel4/EXT_CHC-
- U1 pad 40: /Frontend/ADCChannel7/EXT_CHC+ -> /Frontend/ADCChannel4/EXT_CHB-
- U1 pad 41: /Frontend/ADCChannel7/EXT_CHB- -> /Frontend/ADCChannel4/EXT_CHB+
- U1 pad 42: /Frontend/ADCChannel7/EXT_CHB+ -> /Frontend/ADCChannel4/EXT_CHC+
- U1 pad 43: /Frontend/ADCChannel7/EXT_CHA- -> /Frontend/ADCChannel4/EXT_CHA-
- U1 pad 44: /Frontend/ADCChannel7/EXT_CHA+ -> /Frontend/ADCChannel4/EXT_CHA+
- U1 pad 49: /Frontend/ADCChannel3/EXT_CHD- -> /Frontend/ADCChannel5/EXT_CHD-
- U1 pad 50: /Frontend/ADCChannel3/EXT_CHD+ -> /Frontend/ADCChannel5/EXT_CHD+
- U1 pad 51: /Frontend/ADCChannel3/EXT_CHC- -> /Frontend/ADCChannel5/EXT_CHC-
- U1 pad 52: /Frontend/ADCChannel3/EXT_CHC+ -> /Frontend/ADCChannel5/EXT_CHB-
- U1 pad 53: /Frontend/ADCChannel3/EXT_CHB- -> /Frontend/ADCChannel5/EXT_CHB+
- U1 pad 54: /Frontend/ADCChannel3/EXT_CHB+ -> /Frontend/ADCChannel5/EXT_CHC+
- U1 pad 55: /Frontend/ADCChannel3/EXT_CHA- -> /Frontend/ADCChannel5/EXT_CHA-
- U1 pad 56: /Frontend/ADCChannel3/EXT_CHA+ -> /Frontend/ADCChannel5/EXT_CHA+
- U1 pad 64: /Frontend/ADCChannel6/EXT_CHC+ -> /Frontend/ADCChannel6/EXT_CHB-
- U1 pad 65: /Frontend/ADCChannel6/EXT_CHB- -> /Frontend/ADCChannel6/EXT_CHB+
- U1 pad 66: /Frontend/ADCChannel6/EXT_CHB+ -> /Frontend/ADCChannel6/EXT_CHC+
- U1 pad 73: /Frontend/ADCChannel4/EXT_CHD- -> /Frontend/ADCChannel7/EXT_CHD-
- U1 pad 74: /Frontend/ADCChannel4/EXT_CHD+ -> /Frontend/ADCChannel7/EXT_CHD+
- U1 pad 75: /Frontend/ADCChannel4/EXT_CHC- -> /Frontend/ADCChannel7/EXT_CHC-
- U1 pad 76: /Frontend/ADCChannel4/EXT_CHC+ -> /Frontend/ADCChannel7/EXT_CHB-
- U1 pad 77: /Frontend/ADCChannel4/EXT_CHB- -> /Frontend/ADCChannel7/EXT_CHB+
- U1 pad 78: /Frontend/ADCChannel4/EXT_CHB+ -> /Frontend/ADCChannel7/EXT_CHC+
- U1 pad 79: /Frontend/ADCChannel4/EXT_CHA- -> /Frontend/ADCChannel7/EXT_CHA-
- U1 pad 80: /Frontend/ADCChannel4/EXT_CHA+ -> /Frontend/ADCChannel7/EXT_CHA+
- U1 pad 85: /Frontend/ADCChannel5/EXT_CHD- -> /Frontend/ADCChannel8/EXT_CHD-
- U1 pad 86: /Frontend/ADCChannel5/EXT_CHD+ -> /Frontend/ADCChannel8/EXT_CHD+
- U1 pad 87: /Frontend/ADCChannel5/EXT_CHC- -> /Frontend/ADCChannel8/EXT_CHC-
- U1 pad 88: /Frontend/ADCChannel5/EXT_CHC+ -> /Frontend/ADCChannel8/EXT_CHB-
- U1 pad 89: /Frontend/ADCChannel5/EXT_CHB- -> /Frontend/ADCChannel8/EXT_CHB+
- U1 pad 90: /Frontend/ADCChannel5/EXT_CHB+ -> /Frontend/ADCChannel8/EXT_CHC+
- U1 pad 91: /Frontend/ADCChannel5/EXT_CHA- -> /Frontend/ADCChannel8/EXT_CHA-
- U1 pad 92: /Frontend/ADCChannel5/EXT_CHA+ -> /Frontend/ADCChannel8/EXT_CHA+
Routing:
- net (no net): track 255.8 -> 199.1 mm, vias 31 -> 0
- net /Frontend/ADCChannel8/EXT_CHA-: track 0.00 -> 36.7 mm
- net /Frontend/ADCChannel8/EXT_CHA+: track 0.00 -> 35.8 mm
- net /Frontend/ADCChannel8/EXT_CHB+: track 0.00 -> 35.6 mm
- net /Frontend/ADCChannel8/EXT_CHB-: track 0.00 -> 33.2 mm
- net /Frontend/ADCChannel8/EXT_CHD-: track 0.00 -> 33.0 mm
- net /Frontend/ADCChannel8/EXT_CHC-: track 0.00 -> 32.6 mm
- net /Frontend/ADCChannel2/EXT_CHD-: track 0.00 -> 31.9 mm
- net /Frontend/ADCChannel7/EXT_CHB+: track 0.00 -> 31.8 mm
- net /Frontend/ADCChannel7/EXT_CHA-: track 0.00 -> 31.8 mm
- net /Frontend/ADCChannel8/EXT_CHC+: track 0.00 -> 31.5 mm, vias 0 -> 2
- net /Frontend/ADCChannel7/EXT_CHA+: track 0.00 -> 31.4 mm
- net /Frontend/ADCChannel8/EXT_CHD+: track 0.00 -> 31.3 mm
- net /Frontend/ADCChannel7/EXT_CHD-: track 0.00 -> 31.0 mm
- net /Frontend/ADCChannel7/EXT_CHC-: track 0.00 -> 30.4 mm
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
Commit message: Set proper hysterisis feedback in fan control
Parts:
- added P6: FAN, Socket_Strips:Socket_Strip_Straight_1x02, F.Cu at (21.8, 0.15)
- added Q1: Q_NPN_BCE, Housings_SOT-23_SOT-143_TSOT-6:SOT-23, F.Cu at (14.1, 8.76)
- added R53: 10k, Resistors_SMD:R_0603, F.Cu at (-1.00, 9.30)
- added R54: 10k, Resistors_SMD:R_0603, F.Cu at (-1.00, 11.2)
- added R55: Rf, Resistors_SMD:R_0603, F.Cu at (8.45, 6.10)
- added R56: 253R, Resistors_SMD:R_0603, F.Cu at (10.8, 9.08)
- added RV1: 10k, extras:SM31TW+0805, F.Cu at (2.50, 6.25)
- added TH1: 10k Thermistor, Resistors_SMD:R_0603, F.Cu at (4.05, 15.7)
- added U24: MCP65R41, Housings_SOT-23_SOT-143_TSOT-6:SOT-23-6, F.Cu at (7.30, 8.85)
- moved C7 0.10 mm to (116.1, 57.9)
- moved C10 0.10 mm to (118.1, 57.9)
- moved C23 0.09 mm to (243.8, 58.2)
- moved C24 0.09 mm to (245.6, 58.2)
- moved C37 0.09 mm to (198.2, 57.9)
- moved C40 0.09 mm to (196.2, 57.9)
- moved C13 0.08 mm to (175.8, 57.9)
- moved C16 0.08 mm to (177.8, 57.9)
- moved C19 0.06 mm to (157.8, 57.9)
- moved C22 0.06 mm to (155.8, 57.9)
Connections:
- P3 pad 11: (no net) -> 5Vdig
- P3 pad 16: GNDdig -> GND
- P3 pad 17: GNDdig -> GND
- P3 pad 18: GNDdig -> GND
- P3 pad 19: GNDdig -> GND
- P3 pad 20: GNDdig -> GND
- P3 pad 9: GNDdig -> GND
Routing:
- net (no net): track 199.1 -> 14.2 mm

Commit message: Adds case and board outline
Parts:
- R55: value Rf -> 50k; footprint Resistors_SMD:R_0603 -> Resistors_SMD:R_0805
- moved P6 9.85 mm to (21.8, 10.0)
- moved R55 1.20 mm to (9.22, 5.18)
Connections:
- U24 pad 6: 5Vdig -> 3V3dig
Other:
- board outline added: 160 x 160 mm
Changed lines of the file:
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@@
   (general
     (links 1191)
-    (no_connects 650)
+    (no_connects 651)
     (area 0 0 0 0)
     (thickness 1.6)
-    (drawings 2)
+    (drawings 4)
     (tracks 2341)
     (zones 0)
@@
   )
   (module Socket_Strips:Socket_Strip_Straight_1x02 (layer F.Cu)
-    (at 21.79 0.15)
+    (at 21.79 10)
     (descr "Through hole socket strip")
     (tags "socket strip")
@@
   )
   (module Resistors_SMD:R_0603 (layer F.Cu)
-    (at 8.45 6.1 180)
-    (descr "Resistor SMD 0603, reflow soldering, Vishay (see dcrcw.pdf)")
-    (tags "resistor 0603")
-    (attr smd)
-    (fp_text reference R55 (at 0 1.45 180) (layer F.SilkS)
-      (effects (font (size 1 1) (thickness 0.15)))
-    )
-    (fp_text value Rf (at 0 1.9 180) (layer F.Fab)
-      (effects (font (size 1 1) (thickness 0.15)))
-    )
-    (fp_line (start -1.3 -0.8) (end 1.3 -0.8) (layer F.CrtYd) (width 0.05))
-    (fp_line (start -1.3 0.8) (end 1.3 0.8) (layer F.CrtYd) (width 0.05))
-    (fp_line (start -1.3 -0.8) (end -1.3 0.8) (layer F.CrtYd) (width 0.05))
-    (fp_line (start 1.3 -0.8) (end 1.3 0.8) (layer F.CrtYd) (width 0.05))
-    (fp_line (start 0.5 0.675) (end -0.5 0.675) (layer F.SilkS) (width 0.15))
-    (fp_line (start -0.5 -0.675) (end 0.5 -0.675) (layer F.SilkS) (width 0.15))
-    (pad 1 smd rect (at -0.75 0 180) (size 0.5 0.9) (layers F.Cu F.Paste F.Mask)
-      (net 302 "Net-(R55-Pad1)"))
-    (pad 2 smd rect (at 0.75 0 180) (size 0.5 0.9) (layers F.Cu F.Paste F.Mask)
-      (net 303 "Net-(R55-Pad2)"))
-    (model Resistors_SMD.3dshapes/R_0603.wrl
-      (at (xyz 0 0 0))
-      (scale (xyz 1 1 1))
-      (rotate (xyz 0 0 0))
-    )
-  )
-  (module Resistors_SMD:R_0603 (layer F.Cu)
     (at 10.77 9.08 270)
     (descr "Resistor SMD 0603, reflow soldering, Vishay (see dcrcw.pdf)")
@@
       (net 301 "Net-(R54-Pad2)"))
     (pad 6 smd rect (at 1.1 -0.95 180) (size 1.06 0.65) (layers F.Cu F.Paste F.Mask)
-      (net 296 5Vdig))
+      (net 20 3V3dig))
     (pad 5 smd rect (at 1.1 0 180) (size 1.06 0.65) (layers F.Cu F.Paste F.Mask)
       (net 299 "Net-(R53-Pad1)"))
@@
     )
   )
-  (gr_line (start 101.01 59.39) (end 326.89 59.39) (layer Cmts.User) (width 0.02))
-  (gr_line (start 104.85 33.65) (end 250.45 33.65) (angle 90) (layer Cmts.User) (width 0.02))
+  (module Resistors_SMD:R_0805 (layer F.Cu)
+    (at 9.22 5.18 180)
+    (descr "Resistor SMD 0805, reflow soldering, Vishay (see dcrcw.pdf)")
+    (tags "resistor 0805")
+    (attr smd)
+    (fp_text reference R55 (at 0 -2.1 180) (layer F.SilkS)
+      (effects (font (size 1 1) (thickness 0.15)))
+    )
+    (fp_text value 50k (at 0 2.1 180) (layer F.Fab)
+      (effects (font (size 1 1) (thickness 0.15)))
+    )
+    (fp_line (start -1.6 -1) (end 1.6 -1) (layer F.CrtYd) (width 0.05))
+    (fp_line (start -1.6 1) (end 1.6 1) (layer F.CrtYd) (width 0.05))
+    (fp_line (start -1.6 -1) (end -1.6 1) (layer F.CrtYd) (width 0.05))
+    (fp_line (start 1.6 -1) (end 1.6 1) (layer F.CrtYd) (width 0.05))
+    (fp_line (start 0.6 0.875) (end -0.6 0.875) (layer F.SilkS) (width 0.15))
+    (fp_line (start -0.6 -0.875) (end 0.6 -0.875) (layer F.SilkS) (width 0.15))
+    (pad 1 smd rect (at -0.95 0 180) (size 0.7 1.3) (layers F.Cu F.Paste F.Mask)
+      (net 302 "Net-(R55-Pad1)"))
+    (pad 2 smd rect (at 0.95 0 180) (size 0.7 1.3) (layers F.Cu F.Paste F.Mask)
+      (net 303 "Net-(R55-Pad2)"))
+    (model Resistors_SMD.3dshapes/R_0805.wrl
+      (at (xyz 0 0 0))
+      (scale (xyz 1 1 1))
+      (rotate (xyz 0 0 0))
+    )
+  )
+  (gr_line (start 99 5) (end 99 165) (layer Edge.Cuts) (width 0.15))
+  (gr_line (start 259 5) (end 99 5) (layer Edge.Cuts) (width 0.15))
+  (gr_line (start 259 165) (end 259 5) (layer Edge.Cuts) (width 0.15))
+  (gr_line (start 99 165) (end 259 165) (layer Edge.Cuts) (width 0.15))
   (segment (start 300.79 39.05) (end 301.49 39.05) (width 0.1524) (layer Cmts.User) (net 0))
   (segment (start 300.99 38.85) (end 300.79 39.05) (width 0.1524) (layer Cmts.User) (net 0))
