File: DAQCard2015/DAQCard2015.kicad_pcb (KiCad board)
At the start: 4 copper layers, 160 x 160 mm, 186 parts, among them CON1 BARREL_JACK, P1 QTH-090-01-F-D-A, P2 QTH-090-01-F-D-A, P3 miniDIL20, P4 LEMO_EPY.00.250.NTN, P5 LEMO_EPY.00.250.NTN, P6 FAN, Q1 Q_NPN_BCE, SW1 SPST, U1 RJ45x8, U10 AD9219, U11 THS4524IDBTR, U12 AD9219, U13 THS4524IDBTR, U14 AD9219, U15 THS4524IDBTR, U16 AD9219, U17 THS4524IDBTR, U18 AD9219, U19 CDBHD240-G, U2 AD5628, U20 LM1086, U21 APXS002A0X-SRZ, U22 APXS002A0X-SRZ, U23 APXS002A0X-SRZ, U24 MCP65R41, U3 THS4524IDBTR, U4 AD9219, U5 THS4524IDBTR, U6 AD9219, U7 THS4524IDBTR, U8 AD9219, U9 THS4524IDBTR

Commit message: LVDS pins assigned and first round routing finished, work on 3d models
Parts:
- added REF**: MountingHole_2-5mm, Mounting_Holes:MountingHole_2-5mm, F.Cu at (73.1, 171.5)
- added REF**: MountingHole_2-5mm, Mounting_Holes:MountingHole_2-5mm, F.Cu at (73.1, 100.3)
- added REF**: MountingHole_2-5mm, Mounting_Holes:MountingHole_2-5mm, F.Cu at (121.6, 171.6)
- added REF**: MountingHole_2-5mm, Mounting_Holes:MountingHole_2-5mm, F.Cu at (121.6, 100.4)
- moved P4 287.4 mm to (28.7, 163.8), turned to 180 degrees
- moved P3 266.9 mm to (39.7, 151.9), turned to 180 degrees
- moved P5 265.3 mm to (41.9, 163.8), turned to 180 degrees
- moved C2 206.0 mm to (273.9, 143.5)
- moved C3 206.0 mm to (279.9, 140.0)
- moved C54 206.0 mm to (263.4, 182.5)
- moved C55 206.0 mm to (282.9, 178.0)
- moved C66 206.0 mm to (282.6, 103.1)
- moved D1 206.0 mm to (276.4, 185.0)
- moved R1 206.0 mm to (267.9, 188.5)
- moved R52 206.0 mm to (281.9, 132.0)
- moved C1 206.0 mm to (273.8, 76.7)
- moved C53 206.0 mm to (243.5, 64.6)
- moved C56 206.0 mm to (254.4, 119.1)
- moved C57 206.0 mm to (251.0, 141.2)
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Connections:
- P1 pad 0: /ZEM4310/GNDdig -> GND
- P1 pad 100: (no net) -> /Frontend/2D-D
- P1 pad 103: (no net) -> /Frontend/4D-D
- P1 pad 104: (no net) -> /Frontend/1DCO+
- P1 pad 105: (no net) -> /Frontend/4D+D
- P1 pad 106: (no net) -> /Frontend/1DCO-
- P1 pad 109: (no net) -> /Frontend/4D-C
- P1 pad 110: (no net) -> /Frontend/1FCO+
- P1 pad 111: (no net) -> /Frontend/4D+C
- P1 pad 112: (no net) -> /Frontend/1FCO-
- P1 pad 121: (no net) -> /Frontend/4D-B
- P1 pad 122: (no net) -> /Frontend/1D+A
- P1 pad 123: (no net) -> /Frontend/4D+B
- P1 pad 124: (no net) -> /Frontend/1D-A
- P1 pad 127: (no net) -> /Frontend/4D-A
- P1 pad 128: (no net) -> /Frontend/1D+B
- P1 pad 129: (no net) -> /Frontend/4D+A
- P1 pad 130: (no net) -> /Frontend/1D-B
- P1 pad 133: (no net) -> /Frontend/4FCO-
- P1 pad 134: (no net) -> /Frontend/1D+C
- P1 pad 135: (no net) -> /Frontend/4FCO+
- P1 pad 136: (no net) -> /Frontend/1D-C
- P1 pad 139: (no net) -> /Frontend/4DCO-
- P1 pad 140: (no net) -> /Frontend/1D+D
- P1 pad 141: (no net) -> /Frontend/4DCO+
- P1 pad 142: (no net) -> /Frontend/1D-D
- P1 pad 148: /ZEM4310/H2_LVDS_RXn13 -> /ZEM4310/H1_LVDS_RXn13
- P1 pad 154: /ZEM4310/H2_LVDS_RXn13 -> /ZEM4310/H1_LVDS_RXn13
- P1 pad 67: (no net) -> /Frontend/3D-D
- P1 pad 68: (no net) -> /Frontend/2DCO+
- P1 pad 69: (no net) -> /Frontend/3D+D
- P1 pad 70: (no net) -> /Frontend/2DCO-
- P1 pad 73: (no net) -> /Frontend/3D-C
- P1 pad 74: (no net) -> /Frontend/2FCO+
- P1 pad 75: (no net) -> /Frontend/3D+C
- P1 pad 76: (no net) -> /Frontend/2FCO-
- P1 pad 79: (no net) -> /Frontend/3D-B
- P1 pad 80: (no net) -> /Frontend/2D+A
- P1 pad 81: (no net) -> /Frontend/3D+B
- P1 pad 82: (no net) -> /Frontend/2D-A
- P1 pad 85: (no net) -> /Frontend/3D-A
- P1 pad 86: (no net) -> /Frontend/2D+B
- P1 pad 87: (no net) -> /Frontend/3D+A
- P1 pad 88: (no net) -> /Frontend/2D-B
- P1 pad 91: (no net) -> /Frontend/3FCO-
- P1 pad 92: (no net) -> /Frontend/2D+C
- P1 pad 93: (no net) -> /Frontend/3FCO+
- P1 pad 94: (no net) -> /Frontend/2D-C
- P1 pad 97: (no net) -> /Frontend/3DCO-
- P1 pad 98: (no net) -> /Frontend/2D+D
- P1 pad 99: (no net) -> /Frontend/3DCO+
- P2 pad 0: /ZEM4310/GNDdig -> GND
- P2 pad 100: (no net) -> /Frontend/8DCO-
- P2 pad 103: (no net) -> /Frontend/5D-C
- P2 pad 104: (no net) -> /Frontend/8FCO+
- P2 pad 105: (no net) -> /Frontend/5D+C
- P2 pad 106: (no net) -> /Frontend/8FCO-
- P2 pad 109: (no net) -> /Frontend/5D-B
- P2 pad 110: (no net) -> /Frontend/8D+A
- P2 pad 111: (no net) -> /Frontend/5D+B
- P2 pad 112: (no net) -> /Frontend/8D-A
- P2 pad 121: (no net) -> /Frontend/5D-A
- P2 pad 122: (no net) -> /Frontend/8D+B
- P2 pad 123: (no net) -> /Frontend/5D+A
- P2 pad 124: (no net) -> /Frontend/8D-B
- P2 pad 127: (no net) -> /Frontend/5FCO-
- P2 pad 128: (no net) -> /Frontend/8D+C
- P2 pad 129: (no net) -> /Frontend/5FCO+
- P2 pad 130: (no net) -> /Frontend/8D-C
- P2 pad 133: (no net) -> /Frontend/5DCO-
- P2 pad 134: (no net) -> /Frontend/8D+D
- P2 pad 135: (no net) -> /Frontend/5DCO+
- P2 pad 136: (no net) -> /Frontend/8D-D
- P2 pad 139: (no net) -> /Frontend/6D-D
- P2 pad 140: (no net) -> /Frontend/7DCO+
- P2 pad 141: (no net) -> /Frontend/6D+D
- P2 pad 142: (no net) -> /Frontend/7DCO-
- P2 pad 145: (no net) -> /Frontend/6D-C
- P2 pad 146: (no net) -> /Frontend/7FCO+
- P2 pad 147: (no net) -> /Frontend/6D+C
- P2 pad 148: /ZEM4310/H1_LVDS_RXn13 -> /Frontend/7FCO-
- P2 pad 151: (no net) -> /Frontend/6D-B
- P2 pad 152: (no net) -> /Frontend/7D+A
- P2 pad 153: (no net) -> /Frontend/6D+B
- P2 pad 154: /ZEM4310/H1_LVDS_RXn13 -> /Frontend/7D-A
- P2 pad 157: (no net) -> /Frontend/6D-A
- P2 pad 158: (no net) -> /Frontend/7D+B
- P2 pad 159: (no net) -> /Frontend/6D+A
- P2 pad 160: (no net) -> /Frontend/7D-B
- P2 pad 163: (no net) -> /Frontend/6FCO-
- P2 pad 164: (no net) -> /Frontend/7D+C
- P2 pad 165: (no net) -> /Frontend/6FCO+
- P2 pad 166: (no net) -> /Frontend/7D-C
- P2 pad 169: (no net) -> /Frontend/6DCO-
- P2 pad 170: (no net) -> /Frontend/7D+D
- P2 pad 171: (no net) -> /Frontend/6DCO+
- P2 pad 172: (no net) -> /Frontend/7D-D
- P2 pad 97: (no net) -> /Frontend/5D-D
- P2 pad 98: (no net) -> /Frontend/8DCO+
- P2 pad 99: (no net) -> /Frontend/5D+D
- U10 pad 13: (no net) -> /Frontend/8D-D
- U10 pad 14: (no net) -> /Frontend/8D+D
- U10 pad 15: (no net) -> /Frontend/8D-C
- U10 pad 16: (no net) -> /Frontend/8D+C
- U10 pad 17: (no net) -> /Frontend/8D-B
- U10 pad 18: (no net) -> /Frontend/8D+B
- U10 pad 19: (no net) -> /Frontend/8D-A
- U10 pad 20: (no net) -> /Frontend/8D+A
- U10 pad 21: (no net) -> /Frontend/8FCO-
- U10 pad 22: (no net) -> /Frontend/8FCO+
- U10 pad 23: (no net) -> /Frontend/8DCO-
- U10 pad 24: (no net) -> /Frontend/8DCO+
- U12 pad 13: (no net) -> /Frontend/7D-D
- U12 pad 14: (no net) -> /Frontend/7D+D
- U12 pad 15: (no net) -> /Frontend/7D-C
- U12 pad 16: (no net) -> /Frontend/7D+C
- U12 pad 17: (no net) -> /Frontend/7D-B
- U12 pad 18: (no net) -> /Frontend/7D+B
- U12 pad 19: (no net) -> /Frontend/7D-A
- U12 pad 20: (no net) -> /Frontend/7D+A
- U12 pad 21: (no net) -> /Frontend/7FCO-
- U12 pad 22: (no net) -> /Frontend/7FCO+
- U12 pad 23: (no net) -> /Frontend/7DCO-
- U12 pad 24: (no net) -> /Frontend/7DCO+
- U14 pad 13: (no net) -> /Frontend/5D-D
- U14 pad 14: (no net) -> /Frontend/5D+D
- U14 pad 15: (no net) -> /Frontend/5D-C
- U14 pad 16: (no net) -> /Frontend/5D+C
- U14 pad 17: (no net) -> /Frontend/5D-B
- U14 pad 18: (no net) -> /Frontend/5D+B
- U14 pad 19: (no net) -> /Frontend/5D-A
- U14 pad 20: (no net) -> /Frontend/5D+A
- U14 pad 21: (no net) -> /Frontend/5FCO-
- U14 pad 22: (no net) -> /Frontend/5FCO+
- U14 pad 23: (no net) -> /Frontend/5DCO-
- U14 pad 24: (no net) -> /Frontend/5DCO+
- U16 pad 13: (no net) -> /Frontend/6D-D
- U16 pad 14: (no net) -> /Frontend/6D+D
- U16 pad 15: (no net) -> /Frontend/6D-C
- U16 pad 16: (no net) -> /Frontend/6D+C
- U16 pad 17: (no net) -> /Frontend/6D-B
- U16 pad 18: (no net) -> /Frontend/6D+B
- U16 pad 19: (no net) -> /Frontend/6D-A
- U16 pad 20: (no net) -> /Frontend/6D+A
- U16 pad 21: (no net) -> /Frontend/6FCO-
- U16 pad 22: (no net) -> /Frontend/6FCO+
- U16 pad 23: (no net) -> /Frontend/6DCO-
- U16 pad 24: (no net) -> /Frontend/6DCO+
- U18 pad 13: (no net) -> /Frontend/2D-D
- U18 pad 14: (no net) -> /Frontend/2D+D
- U18 pad 15: (no net) -> /Frontend/2D-C
- U18 pad 16: (no net) -> /Frontend/2D+C
- U18 pad 17: (no net) -> /Frontend/2D-B
- U18 pad 18: (no net) -> /Frontend/2D+B
- U18 pad 19: (no net) -> /Frontend/2D-A
- U18 pad 20: (no net) -> /Frontend/2D+A
- U18 pad 21: (no net) -> /Frontend/2FCO-
- U18 pad 22: (no net) -> /Frontend/2FCO+
- U18 pad 23: (no net) -> /Frontend/2DCO-
- U18 pad 24: (no net) -> /Frontend/2DCO+
- U4 pad 13: (no net) -> /Frontend/1D-D
- U4 pad 14: (no net) -> /Frontend/1D+D
- U4 pad 15: (no net) -> /Frontend/1D-C
- U4 pad 16: (no net) -> /Frontend/1D+C
- U4 pad 17: (no net) -> /Frontend/1D-B
- U4 pad 18: (no net) -> /Frontend/1D+B
- U4 pad 19: (no net) -> /Frontend/1D-A
- U4 pad 20: (no net) -> /Frontend/1D+A
- U4 pad 21: (no net) -> /Frontend/1FCO-
- U4 pad 22: (no net) -> /Frontend/1FCO+
- U4 pad 23: (no net) -> /Frontend/1DCO-
- U4 pad 24: (no net) -> /Frontend/1DCO+
- U6 pad 13: (no net) -> /Frontend/4D-D
- U6 pad 14: (no net) -> /Frontend/4D+D
- U6 pad 15: (no net) -> /Frontend/4D-C
- U6 pad 16: (no net) -> /Frontend/4D+C
- U6 pad 17: (no net) -> /Frontend/4D-B
- U6 pad 18: (no net) -> /Frontend/4D+B
- U6 pad 19: (no net) -> /Frontend/4D-A
- U6 pad 20: (no net) -> /Frontend/4D+A
- U6 pad 21: (no net) -> /Frontend/4FCO-
- U6 pad 22: (no net) -> /Frontend/4FCO+
- U6 pad 23: (no net) -> /Frontend/4DCO-
- U6 pad 24: (no net) -> /Frontend/4DCO+
- U8 pad 13: (no net) -> /Frontend/3D-D
- U8 pad 14: (no net) -> /Frontend/3D+D
- U8 pad 15: (no net) -> /Frontend/3D-C
- U8 pad 16: (no net) -> /Frontend/3D+C
- U8 pad 17: (no net) -> /Frontend/3D-B
- U8 pad 18: (no net) -> /Frontend/3D+B
- U8 pad 19: (no net) -> /Frontend/3D-A
- U8 pad 20: (no net) -> /Frontend/3D+A
- U8 pad 21: (no net) -> /Frontend/3FCO-
- U8 pad 22: (no net) -> /Frontend/3FCO+
- U8 pad 23: (no net) -> /Frontend/3DCO-
- U8 pad 24: (no net) -> /Frontend/3DCO+
Routing:
- net /Frontend/1D-D: track 0.00 -> 100.8 mm
- net /Frontend/1D+D: track 0.00 -> 100.1 mm
- net /Frontend/1D-C: track 0.00 -> 98.9 mm
- net /Frontend/1D+C: track 0.00 -> 98.2 mm
- net /Frontend/1D-B: track 0.00 -> 97.0 mm
- net /Frontend/1D+B: track 0.00 -> 96.3 mm
- net /Frontend/1D-A: track 0.00 -> 95.0 mm
- net /Frontend/1D+A: track 0.00 -> 94.1 mm
- net /Frontend/4DCO+: track 0.00 -> 89.2 mm
- net /Frontend/4DCO-: track 0.00 -> 88.4 mm
- net /Frontend/4FCO+: track 0.00 -> 87.2 mm
- net /Frontend/1FCO-: track 0.00 -> 86.6 mm
- net /Frontend/4FCO-: track 0.00 -> 86.5 mm
- net /Frontend/1FCO+: track 0.00 -> 85.9 mm
- net /Frontend/4D+A: track 0.00 -> 85.3 mm
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- added copper zone on GND.Cu, net GND
