File: DAQCard2015/Frontend.sch (KiCad schematic (older format))
At the start: 0 parts

Commit message: Updates to DAQ Card including FPGA card pinout and completion of ADC Stage
Parts:
- added C?: .1uF, symbol C
- added J2, J4, J? (x6): RJ45_LEDS, symbol RJ45_LEDS
- added R?: 2.4k, symbol R
- added R?: 1k, symbol R
- added R?: 100R, symbol R
- added U?: AD5628, symbol AD5628
Connections:
- net labels added: 1ADC_CSB, 1ADC_Vref, 1D+A, 1D+B, 1D+C, 1D+D, 1D-A, 1D-B, 1D-C, 1D-D, 1DCO+, 1DCO-, 1FCO+, 1FCO-, 2ADC_CSB, 2ADC_Vref, 2D+A, 2D+B, 2D+C, 2D+D, 2D-A, 2D-B, 2D-C, 2D-D, 2DCO+, 2DCO-, 2FCO+, 2FCO-, 3ADC_CSB, 3ADC_Vref, 3D+A, 3D+B, 3D+C, 3D+D, 3D-A, 3D-B, 3D-C, 3D-D, 3DCO+, 3DCO-, 3FCO+, 3FCO-, 3V3, 4ADC_CSB, 4ADC_Vref, 4D+A, 4D+B, 4D+C, 4D+D, 4D-A, 4D-B, 4D-C, 4D-D, 4DCO+, 4DCO-, 4FCO+, 4FCO-, 5ADC_CSB, 5ADC_Vref, 5D+A, 5D+B, 5D+C, 5D+D, 5D-A, 5D-B, 5D-C, 5D-D, 5DCO+, 5DCO-, 5FCO+, 5FCO-, 6ADC_CSB, 6ADC_Vref, 6D+A, 6D+B, 6D+C, 6D+D, 6D-A, 6D-B, 6D-C, 6D-D, 6DCO+, 6DCO-, 6FCO+, 6FCO-, 7ADC_CSB, 7ADC_Vref, 7D+A, 7D+B, 7D+C, 7D+D, 7D-A, 7D-B, 7D-C, 7D-D, 7DCO+, 7DCO-, 7FCO+, 7FCO-, 8ADC_CSB, 8ADC_Vref, 8D+A, 8D+B, 8D+C, 8D+D, 8D-A, 8D-B, 8D-C, 8D-D, 8DCO+, 8DCO-, 8FCO+, 8FCO-, ADC_CLK+, ADC_CLK-, ADC_SCLK, ADC_SDIO, GNDdig, RNGDAC_CSB
- wire segments 0 -> 286
Other:
- note added: "1V ref"

Commit message: Adds power circuitry to DAQCard2015
Connections:
- wire segments 286 -> 246
Changed lines of the file:
@@
 3DCO+
 Wire Wire Line
-	1450 1650 4300 1650
-Wire Wire Line
-	4300 1650 7900 1650
-Wire Wire Line
-	7900 1650 11500 1650
-Wire Wire Line
-	11500 1650 15100 1650
-Wire Wire Line
-	15100 1650 17800 1650
+	1450 1650 17800 1650
 Connection ~ 4400 1550
 Connection ~ 8000 1550
@@
 1ADC_CSB
 Wire Wire Line
-	1450 1750 3950 1750
-Wire Wire Line
-	3950 1750 7550 1750
-Wire Wire Line
-	7550 1750 11150 1750
-Wire Wire Line
-	11150 1750 14750 1750
-Wire Wire Line
-	14750 1750 17900 1750
+	1450 1750 17900 1750
 Wire Wire Line
 	3950 1750 3950 2200
 Wire Wire Line
-	1450 1850 3850 1850
-Wire Wire Line
-	3850 1850 7450 1850
-Wire Wire Line
-	7450 1850 11050 1850
-Wire Wire Line
-	11050 1850 14650 1850
-Wire Wire Line
-	14650 1850 18000 1850
+	1450 1850 18000 1850
 Wire Wire Line
 	3850 1850 3850 2200
@@
 Connection ~ 11050 1850
 Wire Wire Line
-	1450 1550 4400 1550
-Wire Wire Line
-	4400 1550 8000 1550
-Wire Wire Line
-	8000 1550 11600 1550
-Wire Wire Line
-	11600 1550 15200 1550
-Wire Wire Line
-	15200 1550 17700 1550
+	1450 1550 17700 1550
 $Sheet
 S 2700 6000 3400 1050
@@
 6DCO+
 Wire Wire Line
-	17800 5450 15100 5450
-Wire Wire Line
-	15100 5450 11500 5450
-Wire Wire Line
-	11500 5450 7900 5450
-Wire Wire Line
-	7900 5450 4300 5450
-Wire Wire Line
-	4300 5450 2650 5450
+	17800 5450 2650 5450
 Connection ~ 8000 5350
 Connection ~ 11600 5350
@@
 Connection ~ 15100 5450
 Wire Wire Line
-	3950 5550 7550 5550
-Wire Wire Line
-	7550 5550 11150 5550
-Wire Wire Line
-	11150 5550 14750 5550
-Wire Wire Line
-	14750 5550 17900 5550
+	3950 5550 17900 5550
 Wire Wire Line
 	3950 5550 3950 6000
 Wire Wire Line
-	3850 5650 7450 5650
-Wire Wire Line
-	7450 5650 11050 5650
-Wire Wire Line
-	11050 5650 14650 5650
-Wire Wire Line
-	14650 5650 18000 5650
+	3850 5650 18000 5650
 Wire Wire Line
 	3850 5650 3850 6000
@@
 Connection ~ 11050 5650
 Wire Wire Line
-	17700 5350 15200 5350
-Wire Wire Line
-	15200 5350 11600 5350
-Wire Wire Line
-	11600 5350 8000 5350
-Wire Wire Line
-	8000 5350 4400 5350
-Wire Wire Line
-	4400 5350 2650 5350
+	17700 5350 2650 5350
 Connection ~ 14750 5550
 Connection ~ 14650 5650
 Wire Wire Line
-	17700 1550 17700 2550
-Wire Wire Line
-	17700 2550 17700 5350
-Wire Wire Line
-	17800 1650 17800 2450
-Wire Wire Line
-	17800 2450 17800 5450
+	17700 1550 17700 5350
+Wire Wire Line
+	17800 1650 17800 5450
 Wire Wire Line
 	17900 5550 17900 1750
@@
 	18700 3400 18850 3400
 Wire Wire Line
-	18700 3100 18700 3150
-Wire Wire Line
-	18700 3150 18700 3400
+	18700 3100 18700 3400
 Wire Wire Line
 	19950 3600 20450 3600
 Wire Wire Line
-	20450 3150 20450 3600
-Wire Wire Line
-	20450 3600 20450 4100
-Wire Wire Line
-	20450 4100 20450 4450
+	20450 4450 20450 3150
 Wire Wire Line
 	20450 3150 18700 3150
@@
 RNGDAC_CSB
 Wire Wire Line
-	18350 3600 18400 3600
-Wire Wire Line
-	18400 3600 18850 3600
+	18350 3600 18850 3600
 Text GLabel 18350 3600 0    60   Input ~ 0
 3V3
@@
 $EndComp
 Wire Wire Line
-	20450 4450 19350 4450
-Wire Wire Line
-	19350 4450 19250 4450
+	19250 4450 20450 4450
 Connection ~ 20450 4100
 $Comp
@@
 $EndComp
 Wire Wire Line
-	18750 4450 18850 4450
-Wire Wire Line
-	18850 4450 18950 4450
-Wire Wire Line
-	18850 4100 18850 4250
-Wire Wire Line
-	18850 4250 18850 4450
-Wire Wire Line
-	18850 4450 18850 4650
+	18750 4450 18950 4450
+Wire Wire Line
+	18850 4100 18850 4650
 Connection ~ 18850 4450
 Wire Wire Line

Commit message: Replaces single ample with 4-channel varients. Greatly reducing part count
Parts:
- gave numbers to parts that had none: 11
- renumbered J4 to J1, J2 to J3
Connections:
- net labels added: 3V3dig
- net labels removed: 3V3
Changed lines of the file:
@@
 $EndSheet
 $Comp
-L RJ45_LEDS J4
+L RJ45_LEDS J1
 U 1 1 55C8CE8F
 P 5350 1000
-F 0 "J4" H 5350 500 50  0000 C CNN
+F 0 "J1" H 5350 500 50  0000 C CNN
 F 1 "RJ45_LEDS" H 5350 1400 50  0000 C CNN
 F 2 "" H 5350 950 60  0000 C CNN
@@
 $EndSheet
 $Comp
-L RJ45_LEDS J2
+L RJ45_LEDS J3
 U 1 1 55C967FF
 P 9000 1000
-F 0 "J2" H 9000 500 50  0000 C CNN
+F 0 "J3" H 9000 500 50  0000 C CNN
 F 1 "RJ45_LEDS" H 9000 1400 50  0000 C CNN
 F 2 "" H 9000 950 60  0000 C CNN
@@
 	8600 1500 8600 2200
 $Comp
-L RJ45_LEDS J?
+L RJ45_LEDS J7
 U 1 1 55C998EB
 P 16200 1000
-F 0 "J?" H 16200 500 50  0000 C CNN
+F 0 "J7" H 16200 500 50  0000 C CNN
 F 1 "RJ45_LEDS" H 16200 1400 50  0000 C CNN
 F 2 "" H 16200 950 60  0000 C CNN
@@
 	15800 1500 15800 2200
 $Comp
-L RJ45_LEDS J?
+L RJ45_LEDS J5
 U 1 1 55C9999D
 P 12600 1000
-F 0 "J?" H 12600 500 50  0000 C CNN
+F 0 "J5" H 12600 500 50  0000 C CNN
 F 1 "RJ45_LEDS" H 12600 1400 50  0000 C CNN
 F 2 "" H 12600 950 60  0000 C CNN
@@
 $EndSheet
 $Comp
-L RJ45_LEDS J?
+L RJ45_LEDS J2
 U 1 1 55CA4948
 P 5350 4800
-F 0 "J?" H 5350 4300 50  0000 C CNN
+F 0 "J2" H 5350 4300 50  0000 C CNN
 F 1 "RJ45_LEDS" H 5350 5200 50  0000 C CNN
 F 2 "" H 5350 4750 60  0000 C CNN
@@
 $EndSheet
 $Comp
-L RJ45_LEDS J?
+L RJ45_LEDS J4
 U 1 1 55CA4972
 P 9000 4800
-F 0 "J?" H 9000 4300 50  0000 C CNN
+F 0 "J4" H 9000 4300 50  0000 C CNN
 F 1 "RJ45_LEDS" H 9000 5200 50  0000 C CNN
 F 2 "" H 9000 4750 60  0000 C CNN
@@
 	8600 5300 8600 6000
 $Comp
-L RJ45_LEDS J?
+L RJ45_LEDS J8
 U 1 1 55CA4980
 P 16200 4800
-F 0 "J?" H 16200 4300 50  0000 C CNN
+F 0 "J8" H 16200 4300 50  0000 C CNN
 F 1 "RJ45_LEDS" H 16200 5200 50  0000 C CNN
 F 2 "" H 16200 4750 60  0000 C CNN
@@
 	15800 5300 15800 6000
 $Comp
-L RJ45_LEDS J?
+L RJ45_LEDS J6
 U 1 1 55CA498E
 P 12600 4800
-F 0 "J?" H 12600 4300 50  0000 C CNN
+F 0 "J6" H 12600 4300 50  0000 C CNN
 F 1 "RJ45_LEDS" H 12600 5200 50  0000 C CNN
 F 2 "" H 12600 4750 60  0000 C CNN
@@
 Connection ~ 14650 1850
 $Comp
-L R R?
+L R R1
 U 1 1 55CA6D67
 P 2500 5400
-F 0 "R?" V 2580 5400 50  0000 C CNN
+F 0 "R1" V 2580 5400 50  0000 C CNN
 F 1 "100R" V 2500 5400 50  0000 C CNN
 F 2 "" V 2430 5400 30  0000 C CNN
@@
 	4050 6000 4050 5300
 $Comp
-L AD5628 U?
+L AD5628 U1
 U 1 1 55C9703E
 P 19400 3750
-F 0 "U?" H 19700 3200 60  0000 C CNN
+F 0 "U1" H 19700 3200 60  0000 C CNN
 F 1 "AD5628" H 19200 4300 60  0000 C CNN
 F 2 "" H 19600 3900 60  0000 C CNN
@@
 	18350 3600 18850 3600
 Text GLabel 18350 3600 0    60   Input ~ 0
-3V3
+3V3dig
 Wire Wire Line
 	3500 2200 3500 2050
@@
 Connection ~ 18400 3600
 $Comp
-L R R?
+L R R2
 U 1 1 55C9BF1B
 P 18600 4450
-F 0 "R?" V 18680 4450 50  0000 C CNN
+F 0 "R2" V 18680 4450 50  0000 C CNN
 F 1 "2.4k" V 18600 4450 50  0000 C CNN
 F 2 "" V 18530 4450 30  0000 C CNN
@@
 $EndComp
 $Comp
-L R R?
+L R R3
 U 1 1 55C9BF9D
 P 19100 4450
-F 0 "R?" V 19180 4450 50  0000 C CNN
+F 0 "R3" V 19180 4450 50  0000 C CNN
 F 1 "1k" V 19100 4450 50  0000 C CNN
 F 2 "" V 19030 4450 30  0000 C CNN
@@
 Connection ~ 20450 4100
 $Comp
-L C C?
+L C C1
 U 1 1 55C9C14B
 P 19100 4650
-F 0 "C?" H 19125 4750 50  0000 L CNN
+F 0 "C1" H 19125 4750 50  0000 L CNN
 F 1 ".1uF" H 19125 4550 50  0000 L CNN
 F 2 "" H 19138 4500 30  0000 C CNN

Commit message: Finishes initial version of schematic(mostly). And adds a whole bunch of new footprints!
Parts:
- removed J1, J2, J3, J4, J5, J6, J7, J8: RJ45_LEDS, symbol RJ45_LEDS
- added U22: RJ45x8, extras:TE_406967-3, symbol RJ45x8
- C1: footprint (none) -> Capacitors_SMD:C_0603
- R1, R2, R3: footprint (none) -> Resistors_SMD:R_0603
- U1: footprint (none) -> Housings_SSOP:TSSOP-16_4.4x5mm_Pitch0.65mm
Connections:
- wire segments 246 -> 310
Other:
- moved on the sheet: C1, R1, R2, R3, U1

Commit message: Updates to DAQCard2015, especially to power systems
Parts:
- added C?: 10uF, symbol C
- added C?: .1uF, symbol C
- added C?: 10000pF, symbol C
- added R?: 2.7k, symbol R
- added R?: 1k, symbol R
Connections:
- net ADCChannel1/EXT_CHB+: now also U22.5; no longer U22.6
- net ADCChannel1/EXT_CHB-: now also U22.4; no longer U22.5
- net ADCChannel1/EXT_CHC+: now also U22.6; no longer U22.4
- net ADC_CLK+: no longer U1.16 (SCLK)
- net ADC_CLK-: no longer U1.15 (DIN)
- net ADC_SCLK: now also U1.16 (SCLK)
- net ADC_SDIO: now also U1.15 (DIN)
- new net 3V3ana: C?.1, C?.1, R?.1
- new net GND: C?.2, C?.2, C?.2, R?.2
- new net Vocm: C?.1, R?.1, R?.2

Commit message: propogate previous changes to other channels and schematic
Parts:
- C1: renamed from C?; footprint (none) -> Capacitors_SMD:C_0805
- C2, C3: renamed from C?; footprint (none) -> Capacitors_SMD:C_0603
- R1, R2: renamed from R?; footprint (none) -> Resistors_SMD:R_0603
- renumbered C1 to C4, R1 to R3, R2 to R4, R3 to R5, U22 to U1, U1 to U2

Commit message: ADC channels wired, fan controller added
Connections:
- net ADCChannel2/EXT_CHA+: now also U1.20; no longer U1.32
- net ADCChannel2/EXT_CHA-: now also U1.19; no longer U1.31
- net ADCChannel2/EXT_CHB+: now also U1.17; no longer U1.30
- net ADCChannel2/EXT_CHB-: now also U1.16; no longer U1.29
- net ADCChannel2/EXT_CHC+: now also U1.18; no longer U1.28
- net ADCChannel2/EXT_CHC-: now also U1.15; no longer U1.27
- net ADCChannel2/EXT_CHD+: now also U1.14; no longer U1.26
- net ADCChannel2/EXT_CHD-: now also U1.13; no longer U1.25
- net ADCChannel3/EXT_CHA+: now also U1.32; no longer U1.56
- net ADCChannel3/EXT_CHA-: now also U1.31; no longer U1.55
- net ADCChannel3/EXT_CHB+: now also U1.29; no longer U1.54
- net ADCChannel3/EXT_CHB-: now also U1.28; no longer U1.53
- net ADCChannel3/EXT_CHC+: now also U1.30; no longer U1.52
- net ADCChannel3/EXT_CHC-: now also U1.27; no longer U1.51
- net ADCChannel3/EXT_CHD+: now also U1.26; no longer U1.50
- net ADCChannel3/EXT_CHD-: now also U1.25; no longer U1.49
- net ADCChannel4/EXT_CHA+: now also U1.44; no longer U1.80
- net ADCChannel4/EXT_CHA-: now also U1.43; no longer U1.79
- net ADCChannel4/EXT_CHB+: now also U1.41; no longer U1.78
- net ADCChannel4/EXT_CHB-: now also U1.40; no longer U1.77
- net ADCChannel4/EXT_CHC+: now also U1.42; no longer U1.76
- net ADCChannel4/EXT_CHC-: now also U1.39; no longer U1.75
- net ADCChannel4/EXT_CHD+: now also U1.38; no longer U1.74
- net ADCChannel4/EXT_CHD-: now also U1.37; no longer U1.73
- net ADCChannel5/EXT_CHA+: now also U1.56; no longer U1.92
- net ADCChannel5/EXT_CHA-: now also U1.55; no longer U1.91
- net ADCChannel5/EXT_CHB+: now also U1.53; no longer U1.90
- net ADCChannel5/EXT_CHB-: now also U1.52; no longer U1.89
- net ADCChannel5/EXT_CHC+: now also U1.54; no longer U1.88
- net ADCChannel5/EXT_CHC-: now also U1.51; no longer U1.87
- net ADCChannel5/EXT_CHD+: now also U1.50; no longer U1.86
- net ADCChannel5/EXT_CHD-: now also U1.49; no longer U1.85
- net ADCChannel6/EXT_CHB+: now also U1.65; no longer U1.66
- net ADCChannel6/EXT_CHB-: now also U1.64; no longer U1.65
- net ADCChannel6/EXT_CHC+: now also U1.66; no longer U1.64
- net ADCChannel7/EXT_CHA+: now also U1.80; no longer U1.44
- net ADCChannel7/EXT_CHA-: now also U1.79; no longer U1.43
- net ADCChannel7/EXT_CHB+: now also U1.77; no longer U1.42
- net ADCChannel7/EXT_CHB-: now also U1.76; no longer U1.41
- net ADCChannel7/EXT_CHC+: now also U1.78; no longer U1.40
- net ADCChannel7/EXT_CHC-: now also U1.75; no longer U1.39
- net ADCChannel7/EXT_CHD+: now also U1.74; no longer U1.38
- net ADCChannel7/EXT_CHD-: now also U1.73; no longer U1.37
- net ADCChannel8/EXT_CHA+: now also U1.92; no longer U1.20
- net ADCChannel8/EXT_CHA-: now also U1.91; no longer U1.19
- net ADCChannel8/EXT_CHB+: now also U1.89; no longer U1.18
- net ADCChannel8/EXT_CHB-: now also U1.88; no longer U1.17
- net ADCChannel8/EXT_CHC+: now also U1.90; no longer U1.16
- net ADCChannel8/EXT_CHC-: now also U1.87; no longer U1.15
- net ADCChannel8/EXT_CHD+: now also U1.86; no longer U1.14
- net ADCChannel8/EXT_CHD-: now also U1.85; no longer U1.13
- net ADC_CLK+: now also R3.2; no longer R3.1
- net ADC_CLK-: now also R3.1; no longer R3.2
Other:
- moved on the sheet: R3, U1B, U1C, U1D, U1E, U1G, U1H

Commit message: Updates to DAQ system including adjusting position of ZEM and adding Control signal outputs
Parts:
- added P?: CONN_02X20_Double, symbol CONN_02X20_Double
Connections:
- net GND: now also P?.35 (P35), P?.36 (P36), P?.39 (P39), P?.40 (P40), P?.75 (P35), P?.76 (P36), P?.79 (P39), P?.80 (P40)
- net Vocm: now also P?.48 (P8), P?.49 (P9), P?.8 (P8), P?.9 (P9)
- new net 5Vdig: P?.10 (P10), P?.11 (P11), P?.50 (P10), P?.51 (P11)
- new net Aref: P?.34 (P34), P?.74 (P34)
- new net CAL: P?.27 (P27), P?.67 (P27)
- new net CS: P?.14 (P14), P?.54 (P14)
- new net IS1: P?.19 (P19), P?.59 (P19)
- new net IS2: P?.18 (P18), P?.58 (P18)
- new net LE: P?.21 (P21), P?.61 (P21)
- new net NULL: P?.22 (P22), P?.62 (P22)
- new net R12: P?.15 (P15), P?.55 (P15)
- new net RBI: P?.12 (P12), P?.52 (P12)
- new net RBO1: P?.28 (P28), P?.68 (P28)
- new net RBO2: P?.29 (P29), P?.69 (P29)
- new net RBO3: P?.30 (P30), P?.70 (P30)
- new net RBO4: P?.31 (P31), P?.71 (P31)
- new net RG: P?.16 (P16), P?.56 (P16)
- new net RPHI1: P?.33 (P33), P?.73 (P33)
- new net RPHI2: P?.32 (P32), P?.72 (P32)
- new net Reset: P?.20 (P20), P?.60 (P20)
- new net SBI: P?.25 (P25), P?.65 (P25)
- new net SCL: P?.38 (P38), P?.78 (P38)
- new net SDA: P?.37 (P37), P?.77 (P37)
- new net SEB: P?.26 (P26), P?.66 (P26)
- new net SPHI1: P?.24 (P24), P?.64 (P24)
- new net SPHI2: P?.23 (P23), P?.63 (P23)
- new net SR: P?.17 (P17), P?.57 (P17)
- new net Vana: P?.4 (P4), P?.44 (P4), P?.45 (P5), P?.5 (P5)
- new net Vbias: P?.1 (P1), P?.41 (P1)
- new net Vdig: P?.46 (P6), P?.47 (P7), P?.6 (P6), P?.7 (P7)
- new net Vthresh: P?.13 (P13), P?.53 (P13)
- no-connect marks 0 -> 4
Other:
- moved on the sheet: C1, C2, C3, C4, R1, R2, R3, R4, R5, U1A, U1B, U1C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
