File: DAQCard2015/Power.sch (KiCad schematic (older format))
At the start: 28 parts, among them CON1 BARREL_JACK, U18 APXS002A0X-SRZ, U19 APXS002A0X-SRZ, U20 APXS002A0X-SRZ, U21 MCP1826

Commit message: Finishes initial version of schematic(mostly). And adds a whole bunch of new footprints!
Parts:
- removed FI1: MH2029-070Y, symbol EMI_FILTER2
- added FB1: FILTER, Resistors_SMD:R_0805, symbol FILTER
- C74: renamed from C82; footprint (none) -> extras:SMD_Cap_8mmDia
- C75: renamed from C83; footprint (none) -> extras:SMD_Cap_8mmDia
- C76: renamed from C84; footprint (none) -> extras:SMD_Cap_8mmDia
- C77: renamed from C85; footprint (none) -> extras:SMD_Cap_3mmDia
- C78: renamed from C86; footprint (none) -> extras:SMD_Cap_3mmDia
- C79: renamed from C87; footprint (none) -> extras:SMD_Cap_3mmDia
- C80: renamed from C88; footprint (none) -> Capacitors_SMD:C_0603
- C81: renamed from C89; footprint (none) -> Capacitors_SMD:C_0603
- C82: renamed from C90; footprint (none) -> Capacitors_SMD:C_0603
- C83: renamed from C91; footprint (none) -> extras:SMD_Cap_8mmDia
- C84: renamed from C92; footprint (none) -> extras:SMD_Cap_8mmDia
- C85: renamed from C93; footprint (none) -> extras:SMD_Cap_8mmDia
- C86: renamed from C94; footprint (none) -> extras:SMD_Cap_8mmDia
- C87: renamed from C95; footprint (none) -> extras:SMD_Cap_8mmDia
- C88: renamed from C96; value CP -> 100uF; footprint (none) -> extras:SMD_Cap_8mmDia
- C89: renamed from C97; value CP -> 10uF; footprint (none) -> extras:SMD_Cap_3mmDia
- CON1: footprint (none) -> Connect:BARREL_JACK
- R60, R61, R62, R63, R64, R65: footprint (none) -> Resistors_SMD:R_0603
- U18, U19, U20: footprint (none) -> extras:APXS002A0X-SRZ
- U21: footprint (none) -> SMD_Packages:SOT-223
Connections:
- net 3V3ana: now also FB1.2
- net 3V3dig: now also FB1.1
- net GNDdig: now also U21.4 (TAB)
Changed lines of the file:
@@
 F 0 "U18" H 2950 1700 60  0000 C CNN
 F 1 "APXS002A0X-SRZ" H 2600 2400 60  0000 C CNN
-F 2 "" H 2250 1400 60  0000 C CNN
+F 2 "extras:APXS002A0X-SRZ" H 2250 1400 60  0001 C CNN
 F 3 "" H 2250 1400 60  0000 C CNN
 	1    2600 2050
@@
 $EndComp
 $Comp
-L CP C82
+L CP C74
 U 1 1 55CC28F2
 P 1500 2050
-F 0 "C82" H 1525 2150 50  0000 L CNN
+F 0 "C74" H 1525 2150 50  0000 L CNN
 F 1 "100uF" H 1525 1950 50  0000 L CNN
-F 2 "" H 1538 1900 30  0000 C CNN
+F 2 "extras:SMD_Cap_8mmDia" H 1538 1900 30  0001 C CNN
 F 3 "" H 1500 2050 60  0000 C CNN
 	1    1500 2050
@@
 $EndComp
 $Comp
-L C C85
+L C C77
 U 1 1 55CC2951
 P 1750 2050
-F 0 "C85" H 1775 2150 50  0000 L CNN
+F 0 "C77" H 1775 2150 50  0000 L CNN
 F 1 "10uF" H 1775 1950 50  0000 L CNN
-F 2 "" H 1788 1900 30  0000 C CNN
+F 2 "extras:SMD_Cap_3mmDia" H 1788 1900 30  0001 C CNN
 F 3 "" H 1750 2050 60  0000 C CNN
 	1    1750 2050
@@
 F 0 "R60" V 3730 1900 50  0000 C CNN
 F 1 "150R" V 3650 1900 50  0000 C CNN
-F 2 "" V 3580 1900 30  0000 C CNN
+F 2 "Resistors_SMD:R_0603" V 3580 1900 30  0001 C CNN
 F 3 "" H 3650 1900 30  0000 C CNN
 	1    3650 1900
@@
 F 0 "R61" V 3730 2500 50  0000 C CNN
 F 1 "5k" V 3650 2500 50  0000 C CNN
-F 2 "" V 3580 2500 30  0000 C CNN
+F 2 "Resistors_SMD:R_0603" V 3580 2500 30  0001 C CNN
 F 3 "" H 3650 2500 30  0000 C CNN
 	1    3650 2500
@@
 $EndComp
 $Comp
-L C C88
+L C C80
 U 1 1 55CC2A89
 P 3650 2200
-F 0 "C88" H 3675 2300 50  0000 L CNN
+F 0 "C80" H 3675 2300 50  0000 L CNN
 F 1 "10nF" H 3675 2100 50  0000 L CNN
-F 2 "" H 3688 2050 30  0000 C CNN
+F 2 "Capacitors_SMD:C_0603" H 3688 2050 30  0001 C CNN
 F 3 "" H 3650 2200 60  0000 C CNN
 	1    3650 2200
@@
 $EndComp
 $Comp
-L C C91
+L C C83
 U 1 1 55CC2AEA
 P 4100 2150
-F 0 "C91" H 4125 2250 50  0000 L CNN
+F 0 "C83" H 4125 2250 50  0000 L CNN
 F 1 "47uF" H 4125 2050 50  0000 L CNN
-F 2 "" H 4138 2000 30  0000 C CNN
+F 2 "extras:SMD_Cap_8mmDia" H 4138 2000 30  0001 C CNN
 F 3 "" H 4100 2150 60  0000 C CNN
 	1    4100 2150
@@
 Connection ~ 1500 2700
 $Comp
-L C C94
+L C C86
 U 1 1 55CC4361
 P 4350 2150
-F 0 "C94" H 4375 2250 50  0000 L CNN
+F 0 "C86" H 4375 2250 50  0000 L CNN
 F 1 "47uF" H 4375 2050 50  0000 L CNN
-F 2 "" H 4388 2000 30  0000 C CNN
+F 2 "extras:SMD_Cap_8mmDia" H 4388 2000 30  0001 C CNN
 F 3 "" H 4350 2150 60  0000 C CNN
 	1    4350 2150
@@
 F 0 "U19" H 2950 3100 60  0000 C CNN
 F 1 "APXS002A0X-SRZ" H 2600 3800 60  0000 C CNN
-F 2 "" H 2250 2800 60  0000 C CNN
+F 2 "extras:APXS002A0X-SRZ" H 2250 2800 60  0001 C CNN
 F 3 "" H 2250 2800 60  0000 C CNN
 	1    2600 3450
@@
 $EndComp
 $Comp
-L CP C83
+L CP C75
 U 1 1 55CC74F7
 P 1500 3450
-F 0 "C83" H 1525 3550 50  0000 L CNN
+F 0 "C75" H 1525 3550 50  0000 L CNN
 F 1 "100uF" H 1525 3350 50  0000 L CNN
-F 2 "" H 1538 3300 30  0000 C CNN
+F 2 "extras:SMD_Cap_8mmDia" H 1538 3300 30  0001 C CNN
 F 3 "" H 1500 3450 60  0000 C CNN
 	1    1500 3450
@@
 $EndComp
 $Comp
-L C C86
+L C C78
 U 1 1 55CC74FD
 P 1750 3450
-F 0 "C86" H 1775 3550 50  0000 L CNN
+F 0 "C78" H 1775 3550 50  0000 L CNN
 F 1 "10uF" H 1775 3350 50  0000 L CNN
-F 2 "" H 1788 3300 30  0000 C CNN
+F 2 "extras:SMD_Cap_3mmDia" H 1788 3300 30  0001 C CNN
 F 3 "" H 1750 3450 60  0000 C CNN
 	1    1750 3450
@@
 F 0 "R62" V 3730 3300 50  0000 C CNN
 F 1 "150R" V 3650 3300 50  0000 C CNN
-F 2 "" V 3580 3300 30  0000 C CNN
+F 2 "Resistors_SMD:R_0603" V 3580 3300 30  0001 C CNN
 F 3 "" H 3650 3300 30  0000 C CNN
 	1    3650 3300
@@
 F 0 "R63" V 3730 3900 50  0000 C CNN
 F 1 "5k" V 3650 3900 50  0000 C CNN
-F 2 "" V 3580 3900 30  0000 C CNN
+F 2 "Resistors_SMD:R_0603" V 3580 3900 30  0001 C CNN
 F 3 "" H 3650 3900 30  0000 C CNN
 	1    3650 3900
@@
 $EndComp
 $Comp
-L C C89
+L C C81
 U 1 1 55CC750F
 P 3650 3600
-F 0 "C89" H 3675 3700 50  0000 L CNN
+F 0 "C81" H 3675 3700 50  0000 L CNN
 F 1 "10nF" H 3675 3500 50  0000 L CNN
-F 2 "" H 3688 3450 30  0000 C CNN
+F 2 "Capacitors_SMD:C_0603" H 3688 3450 30  0001 C CNN
 F 3 "" H 3650 3600 60  0000 C CNN
 	1    3650 3600
@@
 $EndComp
 $Comp
-L C C92
+L C C84
 U 1 1 55CC7515
 P 4100 3550
-F 0 "C92" H 4125 3650 50  0000 L CNN
+F 0 "C84" H 4125 3650 50  0000 L CNN
 F 1 "47uF" H 4125 3450 50  0000 L CNN
-F 2 "" H 4138 3400 30  0000 C CNN
+F 2 "extras:SMD_Cap_8mmDia" H 4138 3400 30  0001 C CNN
 F 3 "" H 4100 3550 60  0000 C CNN
 	1    4100 3550
@@
 Connection ~ 1500 4100
 $Comp
-L C C95
+L C C87
 U 1 1 55CC7546
 P 4350 3550
-F 0 "C95" H 4375 3650 50  0000 L CNN
+F 0 "C87" H 4375 3650 50  0000 L CNN
 F 1 "47uF" H 4375 3450 50  0000 L CNN
-F 2 "" H 4388 3400 30  0000 C CNN
+F 2 "extras:SMD_Cap_8mmDia" H 4388 3400 30  0001 C CNN
 F 3 "" H 4350 3550 60  0000 C CNN
 	1    4350 3550
@@
 F 0 "U20" H 2950 4550 60  0000 C CNN
 F 1 "APXS002A0X-SRZ" H 2600 5250 60  0000 C CNN
-F 2 "" H 2250 4250 60  0000 C CNN
+F 2 "extras:APXS002A0X-SRZ" H 2250 4250 60  0001 C CNN
 F 3 "" H 2250 4250 60  0000 C CNN
 	1    2600 4900
@@
 $EndComp
 $Comp
-L CP C84
+L CP C76
 U 1 1 55CC7C2D
 P 1500 4900
-F 0 "C84" H 1525 5000 50  0000 L CNN
+F 0 "C76" H 1525 5000 50  0000 L CNN
 F 1 "100uF" H 1525 4800 50  0000 L CNN
-F 2 "" H 1538 4750 30  0000 C CNN
+F 2 "extras:SMD_Cap_8mmDia" H 1538 4750 30  0001 C CNN
 F 3 "" H 1500 4900 60  0000 C CNN
 	1    1500 4900
@@
 $EndComp
 $Comp
-L C C87
+L C C79
 U 1 1 55CC7C33
 P 1750 4900
-F 0 "C87" H 1775 5000 50  0000 L CNN
+F 0 "C79" H 1775 5000 50  0000 L CNN
 F 1 "10uF" H 1775 4800 50  0000 L CNN
-F 2 "" H 1788 4750 30  0000 C CNN
+F 2 "extras:SMD_Cap_3mmDia" H 1788 4750 30  0001 C CNN
 F 3 "" H 1750 4900 60  0000 C CNN
 	1    1750 4900
@@
 F 0 "R64" V 3730 4750 50  0000 C CNN
 F 1 "220R" V 3650 4750 50  0000 C CNN
-F 2 "" V 3580 4750 30  0000 C CNN
+F 2 "Resistors_SMD:R_0603" V 3580 4750 30  0001 C CNN
 F 3 "" H 3650 4750 30  0000 C CNN
 	1    3650 4750
@@
 F 0 "R65" V 3730 5350 50  0000 C CNN
 F 1 "2.22k" V 3650 5350 50  0000 C CNN
-F 2 "" V 3580 5350 30  0000 C CNN
+F 2 "Resistors_SMD:R_0603" V 3580 5350 30  0001 C CNN
 F 3 "" H 3650 5350 30  0000 C CNN
 	1    3650 5350
@@
 $EndComp
 $Comp
-L C C90
+L C C82
 U 1 1 55CC7C45
 P 3650 5050
-F 0 "C90" H 3675 5150 50  0000 L CNN
+F 0 "C82" H 3675 5150 50  0000 L CNN
 F 1 "3900pF" H 3675 4950 50  0000 L CNN
-F 2 "" H 3688 4900 30  0000 C CNN
+F 2 "Capacitors_SMD:C_0603" H 3688 4900 30  0001 C CNN
 F 3 "" H 3650 5050 60  0000 C CNN
 	1    3650 5050
@@
 $EndComp
 $Comp
-L C C93
+L C C85
 U 1 1 55CC7C4B
 P 4100 4950
-F 0 "C93" H 4125 5050 50  0000 L CNN
+F 0 "C85" H 4125 5050 50  0000 L CNN
 F 1 "47uF" H 4125 4850 50  0000 L CNN
-F 2 "" H 4138 4800 30  0000 C CNN
+F 2 "extras:SMD_Cap_8mmDia" H 4138 4800 30  0001 C CNN
 F 3 "" H 4100 4950 60  0000 C CNN
 	1    4100 4950
@@
 Text GLabel 1200 5550 0    60   Input ~ 0
 GNDdig
-$Comp
-L EMI_FILTER2 FI1
-U 1 1 55CCBDB6
-P 1900 6500
-F 0 "FI1" H 1900 6600 50  0000 C CNN
-F 1 "MH2029-070Y" H 1950 6350 50  0000 L CNN
-F 2 "" H 1900 6500 60  0000 C CNN
-F 3 "" H 1900 6500 60  0001 C CNN
-	1    1900 6500
-	1    0    0    -1
-$EndComp
 Text GLabel 1550 6500 0    60   Input ~ 0
 3V3dig
 Text GLabel 2250 6500 2    60   Input ~ 0
 3V3ana
-Text GLabel 1900 6750 3    60   Input ~ 0
-GNDdig
 $Comp
 L MCP1826 U21
@@
 F 0 "U21" H 3450 6950 60  0000 C CNN
 F 1 "MCP1826" V 3850 6900 60  0000 C CNN
-F 2 "" H 3650 6700 60  0000 C CNN
+F 2 "SMD_Packages:SOT-223" H 3650 6700 60  0001 C CNN
 F 3 "" H 3650 6700 60  0000 C CNN
 	1    3650 6700
@@
 F 0 "CON1" H 6200 1200 60  0000 C CNN
 F 1 "BARREL_JACK" H 6200 750 60  0000 C CNN
-F 2 "" H 6200 950 60  0000 C CNN
+F 2 "Connect:BARREL_JACK" H 6200 950 60  0001 C CNN
 F 3 "" H 6200 950 60  0000 C CNN
 	1    6200 950
@@
 	6600 1450 7700 1450
 $Comp
-L CP C96
+L CP C88
 U 1 1 55CD0228
 P 6950 1150
-F 0 "C96" H 6975 1250 50  0000 L CNN
-F 1 "CP" H 6975 1050 50  0000 L CNN
-F 2 "" H 6988 1000 30  0000 C CNN
+F 0 "C88" H 6975 1250 50  0000 L CNN
+F 1 "100uF" H 6975 1050 50  0000 L CNN
+F 2 "extras:SMD_Cap_8mmDia" H 6988 1000 30  0001 C CNN
 F 3 "" H 6950 1150 60  0000 C CNN
 	1    6950 1150
@@
 $EndComp
 $Comp
-L CP C97
+L CP C89
 U 1 1 55CD029E
 P 7200 1150
-F 0 "C97" H 7225 1250 50  0000 L CNN
-F 1 "CP" H 7225 1050 50  0000 L CNN
-F 2 "" H 7238 1000 30  0000 C CNN
+F 0 "C89" H 7225 1250 50  0000 L CNN
+F 1 "10uF" H 7225 1050 50  0000 L CNN
+F 2 "extras:SMD_Cap_3mmDia" H 7238 1000 30  0001 C CNN
 F 3 "" H 7200 1150 60  0000 C CNN
 	1    7200 1150
@@
 NoConn ~ 2000 3600
 NoConn ~ 2000 2200
+Wire Wire Line
+	3350 6350 3000 6350
+Wire Wire Line
+	3000 6350 3000 7000
+Wire Wire Line
+	3000 7000 3650 7000
+Connection ~ 3650 7000
+$Comp
+L FILTER FB1
+U 1 1 55CC0AC4
+P 1900 6500
+F 0 "FB1" H 1900 6650 50  0000 C CNN
+F 1 "FILTER" H 1900 6400 50  0000 C CNN
+F 2 "Resistors_SMD:R_0805" H 1900 6500 60  0001 C CNN
+F 3 "" H 1900 6500 60  0000 C CNN
+	1    1900 6500
+	1    0    0    -1
+$EndComp
 $EndSCHEMATC

Commit message: Adds a more-or-less complete BOM to DAQ Card
Parts:
- C80, C81: value 10nF -> 10000pF
Changed lines of the file:
@@
 P 3650 2200
 F 0 "C80" H 3675 2300 50  0000 L CNN
-F 1 "10nF" H 3675 2100 50  0000 L CNN
+F 1 "10000pF" H 3675 2100 50  0000 L CNN
 F 2 "Capacitors_SMD:C_0603" H 3688 2050 30  0001 C CNN
 F 3 "" H 3650 2200 60  0000 C CNN
@@
 P 3650 3600
 F 0 "C81" H 3675 3700 50  0000 L CNN
-F 1 "10nF" H 3675 3500 50  0000 L CNN
+F 1 "10000pF" H 3675 3500 50  0000 L CNN
 F 2 "Capacitors_SMD:C_0603" H 3688 3450 30  0001 C CNN
 F 3 "" H 3650 3600 60  0000 C CNN

Commit message: Updates to DAQCard2015, especially to power systems
Parts:
- removed C89: 10uF, extras:SMD_Cap_3mmDia, symbol CP
- removed U21: MCP1826, SMD_Packages:SOT-223, symbol MCP1826
- added C89, C90: 10uF, symbol C
- added D1: LED, LEDs:LED-1206, symbol LED
- added R66: 150R, Resistors_SMD:R_0603, symbol R
- added SW1: SPST, extras:Switch_ES02MSABE, symbol SPST
- added U21: CDBHD240-G, extras:mini-DIP4, symbol CDBHD240-G
- added U23: LM1086, extras:TO-263-4, symbol LM1086
- C77, C78, C79: footprint extras:SMD_Cap_3mmDia -> Capacitors_SMD:C_0805
Connections:
- net 5Vdig: now also C74.1, C75.1, C76.1, C77.1, C78.1, C79.1, U18.2 (VIN), U19.2 (VIN), U20.2 (VIN), C90.1, R66.1, U23.2 (OUT), U23.4 (PAD)
- net GNDdig: no longer C88.2, CON1.2, CON1.3
- removed net 5Vraw: C74.1, C75.1, C76.1, C77.1, C78.1, C79.1, C88.1, CON1.1, U18.2 (VIN), U19.2 (VIN), U20.2 (VIN)
- new net: CON1.1, SW1.1
- new net: CON1.2, CON1.3, U21.3 (~~)
- new net: C88.1, C89.1, U21.1 (+), U23.3 (IN)
- new net: SW1.2, U21.4 (~~)
- new net: D1.2 (A), R66.2
- new net GND: C88.2, C89.2, C90.2, D1.1 (K), U21.2 (-), U23.1 (GND)
Other:
- note added: "Power Indicator LED"
- note added: "Shoot for ~~10W DC supply >=7V"
- note removed: "Shoot for ~~10W DC supply @ 5V"
- moved on the sheet: C74, C75, C76, C77, C78, C79, C80, C81, C82, C83, C84, C85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
