File: DAQCard2015/ADCChannel6.sch (KiCad schematic (older format))
At the start: 17 parts, among them U15 THS4524IDBTR, U16 AD9219

Commit message: annotates parts for new build-management tool
Parts:
- C41, C42, C43, C45, C46, C69: Digikey (none) -> 445-1316-1-ND; digipart 445-1316-1-ND -> (none)
- C44: Digikey (none) -> 445-1420-1-ND; digipart 445-1420-1-ND -> (none)
- R36, R37, R38, R39: Digikey (none) -> P107HCT-ND; digipart P107HCT-ND -> (none)
- R40: Digikey (none) -> P10.0KHCT-ND; digipart P10.0KHCT-ND -> (none)
- RP19: Digikey (none) -> RHM1564CT-ND; digipart RHM1564CT-ND -> (none)
- RP20, RP21: Digikey (none) -> RHM1336CT-ND; digipart RHM1336CT-ND -> (none)
- U15: Digikey (none) -> 296-24315-1-ND; digipart 296-24315-1-ND -> (none)
- U16: Digikey (none) -> AD9219ABCPZ-40-ND; digipart AD9219ABCPZ-40-ND -> (none)
Changed lines of the file:
@@
 EESchema Schematic File Version 2
+LIBS:DAQCard2015-rescue
 LIBS:power
 LIBS:device
@@
 F 2 "extras:QFN-48-1EP" H 8650 3700 60  0001 C CNN
 F 3 "" H 8650 3700 60  0000 C CNN
-F 4 "AD9219ABCPZ-40-ND" H 9050 3700 60  0001 C CNN "digipart"
+F 4 "AD9219ABCPZ-40-ND" H 9050 3700 60  0001 C CNN "Digikey"
 	1    9050 3700
 	1    0    0    -1
@@
 F 2 "Capacitors_SMD:C_0603" H 7588 3500 30  0001 C CNN
 F 3 "" H 7550 3650 60  0000 C CNN
-F 4 "445-1316-1-ND" H 7550 3650 60  0001 C CNN "digipart"
+F 4 "445-1316-1-ND" H 7550 3650 60  0001 C CNN "Digikey"
 	1    7550 3650
 	0    1    1    0
@@
 F 2 "Capacitors_SMD:C_0603" H 7588 3800 30  0001 C CNN
 F 3 "" H 7550 3950 60  0000 C CNN
-F 4 "445-1316-1-ND" H 7550 3950 60  0001 C CNN "digipart"
+F 4 "445-1316-1-ND" H 7550 3950 60  0001 C CNN "Digikey"
 	1    7550 3950
 	0    1    1    0
@@
 F 2 "Capacitors_SMD:C_0603" H 9338 1600 30  0001 C CNN
 F 3 "" H 9300 1750 60  0000 C CNN
-F 4 "445-1316-1-ND" H 9300 1750 60  0001 C CNN "digipart"
+F 4 "445-1316-1-ND" H 9300 1750 60  0001 C CNN "Digikey"
 	1    9300 1750
 	0    1    1    0
@@
 F 2 "Capacitors_SMD:C_0603" H 8638 1600 30  0001 C CNN
 F 3 "" H 8600 1750 60  0000 C CNN
-F 4 "445-1316-1-ND" H 8600 1750 60  0001 C CNN "digipart"
+F 4 "445-1316-1-ND" H 8600 1750 60  0001 C CNN "Digikey"
 	1    8600 1750
 	0    1    1    0
@@
 F 2 "Capacitors_SMD:C_0603" H 8988 1500 30  0001 C CNN
 F 3 "" H 8950 1650 60  0000 C CNN
-F 4 "445-1316-1-ND" H 8950 1650 60  0001 C CNN "digipart"
+F 4 "445-1316-1-ND" H 8950 1650 60  0001 C CNN "Digikey"
 	1    8950 1650
 	0    1    1    0
@@
 F 2 "Resistors_SMD:R_0603" V 9830 1950 30  0001 C CNN
 F 3 "" H 9900 1950 30  0000 C CNN
-F 4 "P10.0KHCT-ND" V 9900 1950 60  0001 C CNN "digipart"
+F 4 "P10.0KHCT-ND" V 9900 1950 60  0001 C CNN "Digikey"
 	1    9900 1950
 	0    1    1    0
@@
 F 2 "extras:TSSOP-38_4.4x9.7mm_Pitch0.5mm" H 4600 3800 60  0001 C CNN
 F 3 "" H 4600 3800 60  0000 C CNN
-F 4 "296-24315-1-ND" H 4400 3700 60  0001 C CNN "digipart"
+F 4 "296-24315-1-ND" H 4400 3700 60  0001 C CNN "Digikey"
 	1    4400 3700
 	1    0    0    -1
@@
 F 2 "Resistors_SMD:R_0603" V 1780 4350 30  0001 C CNN
 F 3 "" H 1850 4350 30  0000 C CNN
-F 4 "P107HCT-ND" V 1850 4350 60  0001 C CNN "digipart"
+F 4 "P107HCT-ND" V 1850 4350 60  0001 C CNN "Digikey"
 	1    1850 4350
 	1    0    0    -1
@@
 F 2 "Resistors_SMD:R_0603" V 1780 3850 30  0001 C CNN
 F 3 "" H 1850 3850 30  0000 C CNN
-F 4 "P107HCT-ND" V 1850 3850 60  0001 C CNN "digipart"
+F 4 "P107HCT-ND" V 1850 3850 60  0001 C CNN "Digikey"
 	1    1850 3850
 	1    0    0    -1
@@
 F 2 "Resistors_SMD:R_0603" V 1780 3350 30  0001 C CNN
 F 3 "" H 1850 3350 30  0000 C CNN
-F 4 "P107HCT-ND" V 1850 3350 60  0001 C CNN "digipart"
+F 4 "P107HCT-ND" V 1850 3350 60  0001 C CNN "Digikey"
 	1    1850 3350
 	1    0    0    -1
@@
 F 2 "Resistors_SMD:R_0603" V 1780 2850 30  0001 C CNN
 F 3 "" H 1850 2850 30  0000 C CNN
-F 4 "P107HCT-ND" V 1850 2850 60  0001 C CNN "digipart"
+F 4 "P107HCT-ND" V 1850 2850 60  0001 C CNN "Digikey"
 	1    1850 2850
 	1    0    0    -1
@@
 F 2 "extras:R4-MNR04" H 4250 5150 60  0001 C CNN
 F 3 "" H 4250 5150 60  0000 C CNN
-F 4 "RHM1336CT-ND" H 4250 5150 60  0001 C CNN "digipart"
+F 4 "RHM1336CT-ND" H 4250 5150 60  0001 C CNN "Digikey"
 	1    4250 5150
 	1    0    0    -1
@@
 F 2 "extras:R4-MNR04" H 4300 2450 60  0001 C CNN
 F 3 "" H 4300 2450 60  0000 C CNN
-F 4 "RHM1336CT-ND" H 4300 2450 60  0001 C CNN "digipart"
+F 4 "RHM1336CT-ND" H 4300 2450 60  0001 C CNN "Digikey"
 	1    4300 2450
 	1    0    0    -1
@@
 F 2 "extras:R8_MNR18" H 2750 3600 60  0001 C CNN
 F 3 "" H 2750 3600 60  0000 C CNN
-F 4 "RHM1564CT-ND" H 2750 3600 60  0001 C CNN "digipart"
+F 4 "RHM1564CT-ND" H 2750 3600 60  0001 C CNN "Digikey"
 	1    2750 3600
 	1    0    0    -1
@@
 F 2 "Capacitors_SMD:C_0805" H 8988 1300 30  0001 C CNN
 F 3 "" H 8950 1450 60  0000 C CNN
-F 4 "445-1420-1-ND" H 8950 1450 60  0001 C CNN "digipart"
+F 4 "445-1420-1-ND" H 8950 1450 60  0001 C CNN "Digikey"
 	1    8950 1450
 	0    -1   -1   0
@@
 F 2 "Capacitors_SMD:C_0603" H 4438 5350 30  0001 C CNN
 F 3 "" H 4400 5500 60  0000 C CNN
-F 4 "445-1316-1-ND" H 4400 5500 60  0001 C CNN "digipart"
+F 4 "445-1316-1-ND" H 4400 5500 60  0001 C CNN "Digikey"
 	1    4400 5500
 	0    1    1    0
