File: DAQCard2015/ZEM4310.sch (KiCad schematic (older format))
At the start: 2 parts, among them P1 QTH-090-01-F-D-A, P2 QTH-090-01-F-D-A

Commit message: Update V1.0 of DAQ Board Includes LED Driver for RJ45 Port, repositioning of JTAG
Connections:
- net EXT_TRG: now also P2.87; no longer P2.81
- net IS1: now also P2.81; no longer P1.145
- net Reset: now also P2.85; no longer P1.147
- net RJ45_LED_LATCH: now reaches P2.115
- net RJ45_LED_CLK: now reaches P2.116
- net RJ45_LED_BLANK: now reaches P2.117
- net RJ45_LED_SDA: now reaches P2.118
- new net NULL: P1.147
Changed lines of the file:
@@
 NoConn ~ 8000 2000
 NoConn ~ 8000 2100
-Text Label 9550 2100 0    60   ~ 0
-+VCCIO4
-Text Label 7950 2200 2    60   ~ 0
-+Y_HSMC_VCCIO
 NoConn ~ 8000 2400
 NoConn ~ 8000 2300
 NoConn ~ 9500 2300
 NoConn ~ 9500 2200
-Text Label 9550 2400 0    60   ~ 0
-+VCCIO5
 NoConn ~ 9500 2500
 NoConn ~ 9500 2600
 NoConn ~ 8000 2600
 NoConn ~ 8000 2700
-Text Label 9550 2700 0    60   ~ 0
-+VCCIO6
 NoConn ~ 8000 2900
 NoConn ~ 8000 3000
 NoConn ~ 9500 2800
 NoConn ~ 9500 2900
-Text Label 9550 3000 0    60   ~ 0
-VREF_BANK4
 NoConn ~ 8000 3200
 NoConn ~ 8000 3300
 NoConn ~ 9500 3100
 NoConn ~ 9500 3200
-Text Label 9550 3300 0    60   ~ 0
-VREF_BANK5
-Text Label 7950 3400 2    60   ~ 0
-VREF_BANK6
-Text Label 9550 3400 0    60   ~ 0
-PLL4_CLKOUTp
 NoConn ~ 8000 3500
-Text Label 9550 3500 0    60   ~ 0
-PLL4_CLKOUTn
 NoConn ~ 8000 3600
 NoConn ~ 9500 3600
-Text Label 9550 3700 0    60   ~ 0
-HSMC_SDA
-Text Label 7950 3800 2    60   ~ 0
-HSMC_SCL
 NoConn ~ 9500 3900
 NoConn ~ 8000 4000
-Text Label 9550 4100 0    60   ~ 0
-CLKOUT0
 NoConn ~ 8000 4300
-Text Label 9550 7000 0    60   ~ 0
-CLKOUT1p
-Text Label 9550 7100 0    60   ~ 0
-CLKOUT1n
-Text Label 7950 7100 2    60   ~ 0
-CLKIN1p
-Text Label 7950 7200 2    60   ~ 0
-CLKIN1n
 Text Notes 2340 10400 1    60   ~ 0
 HSMC  J1
@@
 NoConn ~ 3450 7050
 NoConn ~ 3450 7150
-NoConn ~ 8000 7200
-NoConn ~ 8000 7100
-NoConn ~ 9500 7100
-NoConn ~ 9500 7000
 NoConn ~ 1950 2550
 NoConn ~ 1950 2850
@@
 Text GLabel 3450 3550 2    40   Input ~ 0
 ADC_CLK-
-Text GLabel 3450 8550 2    40   Input ~ 0
+Text GLabel 9500 5300 2    40   Input ~ 0
 IS1
-Text GLabel 3450 8650 2    40   Input ~ 0
+Text GLabel 9500 5500 2    40   Input ~ 0
 Reset
 Text GLabel 3450 8850 2    40   Input ~ 0
@@
 Text GLabel 9500 4300 2    40   Input ~ 0
 LED1
-Text Label 7950 3100 2    60   ~ 0
-Y_HSMC_VS2
-Text Label 7950 2800 2    60   ~ 0
-Y_HSMC_VS1
-Text Label 7950 2500 2    60   ~ 0
-Y_HSMC_VS0
 Text GLabel 1950 3750 0    40   Input ~ 0
 JTAG_TDO
@@
 Text GLabel 8000 4500 0    40   Input ~ 0
 UIO_2
-Text GLabel 9500 5300 2    40   Input ~ 0
+Text GLabel 9500 5600 2    40   Input ~ 0
 EXT_TRG
+Text Label 9550 4100 0    60   ~ 0
+CLKOUT0
+Text Label 7950 3800 2    60   ~ 0
+HSMC_SCL
+Text Label 7950 3400 2    60   ~ 0
+VREF_BANK6
+Text Label 7950 3100 2    60   ~ 0
+Y_HSMC_VS2
+Text Label 7950 2800 2    60   ~ 0
+Y_HSMC_VS1
+Text Label 7950 2500 2    60   ~ 0
+Y_HSMC_VS0
+Text Label 7950 2200 2    60   ~ 0
++Y_HSMC_VCCIO
+Text Label 9550 2100 0    60   ~ 0
++VCCIO4
+Text Label 9550 2400 0    60   ~ 0
++VCCIO5
+Text Label 9550 2700 0    60   ~ 0
++VCCIO6
+Text Label 9550 3000 0    60   ~ 0
+VREF_BANK4
+Text Label 9550 3300 0    60   ~ 0
+VREF_BANK5
+Text Label 9550 3400 0    60   ~ 0
+PLL4_CLKOUTp
+Text Label 9550 3500 0    60   ~ 0
+PLL4_CLKOUTn
+Text Label 9550 3700 0    60   ~ 0
+HSMC_SDA
+NoConn ~ 9500 3700
+NoConn ~ 9500 4100
+NoConn ~ 8000 3800
+NoConn ~ 8000 4200
+Text GLabel 3450 8650 2    40   Input ~ 0
+NULL
+Text GLabel 8000 7100 0    40   Input ~ 0
+RJ45_LED_CLK
+Text GLabel 8000 7200 0    40   Input ~ 0
+RJ45_LED_SDA
+Text GLabel 9500 7100 2    40   Input ~ 0
+RJ45_LED_BLANK
+Text GLabel 9500 7000 2    40   Input ~ 0
+RJ45_LED_LATCH
 $EndSCHEMATC

Commit message: Adds digipart field to all parts that is now used in automatic generation of BOM(see DAQCard2015.html)
Parts:
- P1, P2: digipart (none) -> SAM8195-ND
Changed lines of the file:
@@
 F 2 "extras:QTH-090-XX-X-D-A" H 2700 5850 50  0001 C CNN
 F 3 "DOCUMENTATION" H 2700 5850 50  0001 C CNN
+F 4 "SAM8195-ND" H 2700 5850 60  0001 C CNN "digipart"
 	1    2700 5850
 	1    0    0    -1
@@
 F 2 "extras:QTH-090-XX-X-D-A" H 8750 5800 50  0001 C CNN
 F 3 "DOCUMENTATION" H 8750 5800 50  0001 C CNN
+F 4 "SAM8195-ND" H 8750 5800 60  0001 C CNN "digipart"
 	1    8750 5800
 	1    0    0    -1

Commit message: annotates parts for new build-management tool
Parts:
- P1, P2: Digikey (none) -> SAM8195-ND; digipart SAM8195-ND -> (none)
Changed lines of the file:
@@
 EESchema Schematic File Version 2
+LIBS:DAQCard2015-rescue
 LIBS:power
 LIBS:device
@@
 F 2 "extras:QTH-090-XX-X-D-A" H 2700 5850 50  0001 C CNN
 F 3 "DOCUMENTATION" H 2700 5850 50  0001 C CNN
-F 4 "SAM8195-ND" H 2700 5850 60  0001 C CNN "digipart"
+F 4 "SAM8195-ND" H 2700 5850 60  0001 C CNN "Digikey"
 	1    2700 5850
 	1    0    0    -1
@@
 F 2 "extras:QTH-090-XX-X-D-A" H 8750 5800 50  0001 C CNN
 F 3 "DOCUMENTATION" H 8750 5800 50  0001 C CNN
-F 4 "SAM8195-ND" H 8750 5800 60  0001 C CNN "digipart"
+F 4 "SAM8195-ND" H 8750 5800 60  0001 C CNN "Digikey"
 	1    8750 5800
 	1    0    0    -1
